File: pico-hat-stepper/assembly.kicad_sch (KiCad schematic)
At the start: 8 parts

Commit message: tmc5160_featherwing -> pico-hat-stepper
Other:
- title: tmc5160_featherwing -> pico-hat-stepper
Changed lines of the file:
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@@
   (paper "A4")
   (title_block
-    (title "tmc5160_featherwing")
+    (title "pico-hat-stepper")
     (date "2024-04-16")
     (rev "1.0")
@@
     (pin "1")
     (instances
-      (project "tmc5160_featherwing"
+      (project "pico-hat-stepper"
         (path "/df2b2e89-e055-4140-95de-f1df723db034/0ec4fe58-7f94-4826-b0e2-2bc8f3ffe81e"
           (reference "H1") (unit 1)
@@
     )
     (instances
-      (project "tmc5160_featherwing"
+      (project "pico-hat-stepper"
         (path "/df2b2e89-e055-4140-95de-f1df723db034/0ec4fe58-7f94-4826-b0e2-2bc8f3ffe81e"
           (reference "FID2") (unit 1)
@@
     (pin "1")
     (instances
-      (project "tmc5160_featherwing"
+      (project "pico-hat-stepper"
         (path "/df2b2e89-e055-4140-95de-f1df723db034/0ec4fe58-7f94-4826-b0e2-2bc8f3ffe81e"
           (reference "H3") (unit 1)
@@
     )
     (instances
-      (project "tmc5160_featherwing"
+      (project "pico-hat-stepper"
         (path "/df2b2e89-e055-4140-95de-f1df723db034/0ec4fe58-7f94-4826-b0e2-2bc8f3ffe81e"
           (reference "FID4") (unit 1)
@@
     )
     (instances
-      (project "tmc5160_featherwing"
+      (project "pico-hat-stepper"
         (path "/df2b2e89-e055-4140-95de-f1df723db034/0ec4fe58-7f94-4826-b0e2-2bc8f3ffe81e"
           (reference "FID1") (unit 1)
@@
     (pin "1")
     (instances
-      (project "tmc5160_featherwing"
+      (project "pico-hat-stepper"
         (path "/df2b2e89-e055-4140-95de-f1df723db034/0ec4fe58-7f94-4826-b0e2-2bc8f3ffe81e"
           (reference "H4") (unit 1)
@@
     (pin "1")
     (instances
-      (project "tmc5160_featherwing"
+      (project "pico-hat-stepper"
         (path "/df2b2e89-e055-4140-95de-f1df723db034/0ec4fe58-7f94-4826-b0e2-2bc8f3ffe81e"
           (reference "H2") (unit 1)
@@
     )
     (instances
-      (project "tmc5160_featherwing"
+      (project "pico-hat-stepper"
         (path "/df2b2e89-e055-4140-95de-f1df723db034/0ec4fe58-7f94-4826-b0e2-2bc8f3ffe81e"
           (reference "FID3") (unit 1)
