File: pico-hat-stepper/featherwing.kicad_sch (KiCad schematic)
At the start: 2 parts, among them J6 Conn_01x16_P2.54MM_HeaderHoles, J7 Conn_01x12_P2.54MM_HeaderHoles

Commit message: tmc5160_featherwing -> pico-hat-stepper
Other:
- title: tmc5160_featherwing -> pico-hat-stepper
Changed lines of the file:
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@@
   (paper "A4")
   (title_block
-    (title "tmc5160_featherwing")
+    (title "pico-hat-stepper")
     (date "2024-04-16")
     (rev "1.0")
@@
     (pin "1")
     (instances
-      (project "tmc5160_featherwing"
+      (project "pico-hat-stepper"
         (path "/df2b2e89-e055-4140-95de-f1df723db034/69dff8eb-dcc1-4f17-9e1d-cf8103035e92"
           (reference "J6") (unit 1)
@@
     (pin "4")
     (instances
-      (project "tmc5160_featherwing"
+      (project "pico-hat-stepper"
         (path "/df2b2e89-e055-4140-95de-f1df723db034/69dff8eb-dcc1-4f17-9e1d-cf8103035e92"
           (reference "J7") (unit 1)
