File: pico-hat-stepper/mosfet.kicad_sch (KiCad schematic)
At the start: 2 parts, among them U4 BUK7D36-60EX

Commit message: tmc5160_featherwing -> pico-hat-stepper
Other:
- title: tmc5160_featherwing -> pico-hat-stepper
Changed lines of the file:
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@@
   (paper "A4")
   (title_block
-    (title "tmc5160_featherwing")
+    (title "pico-hat-stepper")
     (date "2024-04-16")
     (rev "1.0")
@@
     (pin "8")
     (instances
-      (project "tmc5160_featherwing"
+      (project "pico-hat-stepper"
         (path "/df2b2e89-e055-4140-95de-f1df723db034/039ac378-5273-4081-85bf-9eb26cb5ed57/166b4ba4-5822-49d8-b309-f52ce04f60b1"
           (reference "U4") (unit 1)
@@
     (pin "1")
     (instances
-      (project "tmc5160_featherwing"
+      (project "pico-hat-stepper"
         (path "/df2b2e89-e055-4140-95de-f1df723db034/039ac378-5273-4081-85bf-9eb26cb5ed57/166b4ba4-5822-49d8-b309-f52ce04f60b1"
           (reference "R10") (unit 1)
