File: pico-hat-stepper/power.kicad_sch (KiCad schematic)
At the start: 14 parts, among them J1 Conn_01x03_P2.54MM_HeaderHoles, J2 Conn_01x02_P1.5MM_Molex_Pico-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, J3 Conn_01x03_P2.54MM_HeaderHoles, J8 HEADER_01X03_JST_SUR_VERTICAL, Q1 MOSFET-N-CH, U1 3.3V_100MA

Commit message: tmc5160_featherwing -> pico-hat-stepper
Other:
- title: tmc5160_featherwing -> pico-hat-stepper
Changed lines of the file:
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@@
   (paper "A4")
   (title_block
-    (title "tmc5160_featherwing")
+    (title "pico-hat-stepper")
     (date "2024-04-16")
     (rev "1.0")
@@
     (pin "3")
     (instances
-      (project "tmc5160_featherwing"
+      (project "pico-hat-stepper"
         (path "/df2b2e89-e055-4140-95de-f1df723db034/c1dd8f61-494c-402f-8e59-08309c64fc3f"
           (reference "J8") (unit 1)
@@
     (pin "1")
     (instances
-      (project "tmc5160_featherwing"
+      (project "pico-hat-stepper"
         (path "/df2b2e89-e055-4140-95de-f1df723db034/c1dd8f61-494c-402f-8e59-08309c64fc3f"
           (reference "C20") (unit 1)
@@
     (pin "3")
     (instances
-      (project "tmc5160_featherwing"
+      (project "pico-hat-stepper"
         (path "/df2b2e89-e055-4140-95de-f1df723db034/c1dd8f61-494c-402f-8e59-08309c64fc3f"
           (reference "J3") (unit 1)
@@
     (pin "1")
     (instances
-      (project "tmc5160_featherwing"
+      (project "pico-hat-stepper"
         (path "/df2b2e89-e055-4140-95de-f1df723db034/c1dd8f61-494c-402f-8e59-08309c64fc3f"
           (reference "R18") (unit 1)
@@
     (pin "2")
     (instances
-      (project "tmc5160_featherwing"
+      (project "pico-hat-stepper"
         (path "/df2b2e89-e055-4140-95de-f1df723db034/c1dd8f61-494c-402f-8e59-08309c64fc3f"
           (reference "D2") (unit 1)
@@
     (pin "1")
     (instances
-      (project "tmc5160_featherwing"
+      (project "pico-hat-stepper"
         (path "/df2b2e89-e055-4140-95de-f1df723db034/c1dd8f61-494c-402f-8e59-08309c64fc3f"
           (reference "C2") (unit 1)
@@
     (pin "1")
     (instances
-      (project "tmc5160_featherwing"
+      (project "pico-hat-stepper"
         (path "/df2b2e89-e055-4140-95de-f1df723db034/c1dd8f61-494c-402f-8e59-08309c64fc3f"
           (reference "J2") (unit 1)
@@
     (pin "3")
     (instances
-      (project "tmc5160_featherwing"
+      (project "pico-hat-stepper"
         (path "/df2b2e89-e055-4140-95de-f1df723db034/c1dd8f61-494c-402f-8e59-08309c64fc3f"
           (reference "J1") (unit 1)
@@
     (pin "3")
     (instances
-      (project "tmc5160_featherwing"
+      (project "pico-hat-stepper"
         (path "/df2b2e89-e055-4140-95de-f1df723db034/c1dd8f61-494c-402f-8e59-08309c64fc3f"
           (reference "U1") (unit 1)
@@
     (pin "1")
     (instances
-      (project "tmc5160_featherwing"
+      (project "pico-hat-stepper"
         (path "/df2b2e89-e055-4140-95de-f1df723db034/c1dd8f61-494c-402f-8e59-08309c64fc3f"
           (reference "Q1") (unit 1)
@@
     (pin "2")
     (instances
-      (project "tmc5160_featherwing"
+      (project "pico-hat-stepper"
         (path "/df2b2e89-e055-4140-95de-f1df723db034/c1dd8f61-494c-402f-8e59-08309c64fc3f"
           (reference "R2") (unit 1)
@@
     (pin "2")
     (instances
-      (project "tmc5160_featherwing"
+      (project "pico-hat-stepper"
         (path "/df2b2e89-e055-4140-95de-f1df723db034/c1dd8f61-494c-402f-8e59-08309c64fc3f"
           (reference "C1") (unit 1)
@@
     (pin "2")
     (instances
-      (project "tmc5160_featherwing"
+      (project "pico-hat-stepper"
         (path "/df2b2e89-e055-4140-95de-f1df723db034/c1dd8f61-494c-402f-8e59-08309c64fc3f"
           (reference "D1") (unit 1)
@@
     (pin "1")
     (instances
-      (project "tmc5160_featherwing"
+      (project "pico-hat-stepper"
         (path "/df2b2e89-e055-4140-95de-f1df723db034/c1dd8f61-494c-402f-8e59-08309c64fc3f"
           (reference "R1") (unit 1)
