File: pico-hat-stepper/pico-hat-stepper.kicad_pcb (KiCad board)
At the start: 2 copper layers, 72 x 22.9 mm, 40 parts, among them J1 Conn_01x03_P2.54MM_HeaderHoles, J2 Conn_01x02_P1.5MM_Molex_Pico-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, J3 Conn_01x03_P2.54MM_HeaderHoles, J4 Conn_01x04_P1.5MM_Molex_Pico-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, J5 Conn_01x02_P1.5MM_Molex_Pico-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, J6 Conn_01x16_P2.54MM_HeaderHoles, J7 Conn_01x12_P2.54MM_HeaderHoles, U1 TMC5160A-WA, U10 3.3V_100MA, U11 MAX6816, U2 BUK7D36-60EX, U3 BUK7D36-60EX, U4 BUK7D36-60EX, U5 BUK7D36-60EX, U6 BUK7D36-60EX, U7 BUK7D36-60EX, U8 BUK7D36-60EX, U9 BUK7D36-60EX, X1 16MHz

Commit message: featherwing -> pico-hat
Connections:
- net /driver_controller/CLOCK renamed /driver-controller/CLOCK
- net /driver_controller/MISO renamed /driver-controller/MISO
- net /driver_controller/MOSI renamed /driver-controller/MOSI
- net /driver_controller/SCK renamed /driver-controller/SCK
- net /driver_controller/mosfet1/DRAIN renamed /driver-controller/mosfet1/DRAIN
- net /driver_controller/mosfet1/GATE renamed /driver-controller/mosfet1/GATE
- net /driver_controller/mosfet1/SOURCE renamed /driver-controller/mosfet1/SOURCE
- net /driver_controller/mosfet2/DRAIN renamed /driver-controller/mosfet2/DRAIN
- net /driver_controller/mosfet2/GATE renamed /driver-controller/mosfet2/GATE
- net /driver_controller/mosfet2/SOURCE renamed /driver-controller/mosfet2/SOURCE
- net /driver_controller/mosfet3/DRAIN renamed /driver-controller/mosfet3/DRAIN
- net /driver_controller/mosfet3/GATE renamed /driver-controller/mosfet3/GATE
- net /driver_controller/mosfet3/SOURCE renamed /driver-controller/mosfet3/SOURCE
- net /driver_controller/mosfet4/DRAIN renamed /driver-controller/mosfet4/DRAIN
- net /driver_controller/mosfet4/GATE renamed /driver-controller/mosfet4/GATE
- net /driver_controller/mosfet4/SOURCE renamed /driver-controller/mosfet4/SOURCE
- net /driver_controller/mosfet5/DRAIN renamed /driver-controller/mosfet5/DRAIN
- net /driver_controller/mosfet5/GATE renamed /driver-controller/mosfet5/GATE
- net /driver_controller/mosfet5/SOURCE renamed /driver-controller/mosfet5/SOURCE
- net /driver_controller/mosfet6/DRAIN renamed /driver-controller/mosfet6/DRAIN
- net /driver_controller/mosfet6/GATE renamed /driver-controller/mosfet6/GATE
- net /driver_controller/mosfet6/SOURCE renamed /driver-controller/mosfet6/SOURCE
- net /driver_controller/mosfet7/DRAIN renamed /driver-controller/mosfet7/DRAIN
- net /driver_controller/mosfet7/GATE renamed /driver-controller/mosfet7/GATE
- net /driver_controller/mosfet7/SOURCE renamed /driver-controller/mosfet7/SOURCE
- net /driver_controller/mosfet8/DRAIN renamed /driver-controller/mosfet8/DRAIN
- net /driver_controller/mosfet8/GATE renamed /driver-controller/mosfet8/GATE
- net /driver_controller/mosfet8/SOURCE renamed /driver-controller/mosfet8/SOURCE
- net /driver_controller/~{CS} renamed /driver-controller/~{CS}
