File: pico-hat-stepper/pico-hat.kicad_sch (KiCad schematic)
At the start: 2 parts, among them J6 Conn_01x16_P2.54MM_HeaderHoles, J7 Conn_01x12_P2.54MM_HeaderHoles

Commit message: Adjust
Parts:
- removed J6: Conn_01x16_P2.54MM_HeaderHoles, Janelia:PinHeader_1x16_P2.54mm_Vertical_Holes, symbol Janelia:Conn_01x16_P2.54MM_HeaderHoles
- removed J7: Conn_01x12_P2.54MM_HeaderHoles, Janelia:PinHeader_1x12_P2.54mm_Vertical_Holes, symbol Janelia:Conn_01x12_P2.54MM_HeaderHoles
Connections:
- no-connect marks 2 -> 0
Changed lines of the file:
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@@
     (company "Howard Hughes Medical Institute")
   )
-  (no_connect (at 102.87 74.93))
-  (no_connect (at 102.87 77.47))
   (wire (pts (xy 43.18 76.2) (xy 45.72 76.2))
     (stroke (width 0) (type default))
@@
   )
   (wire (pts (xy 43.18 60.96) (xy 45.72 60.96))
-    (stroke (width 0) (type default))
-  )
-  (wire (pts (xy 96.52 63.5) (xy 99.06 63.5))
     (stroke (width 0) (type default))
   )
@@
     (effects (font (size 1.27 1.27)) (justify right))
   )
-  (symbol (lib_id "Janelia:Conn_01x16_P2.54MM_HeaderHoles") (at 107.95 92.71 0) (unit 1)
-    (in_bom no) (on_board yes) (dnp no)
-    (property "Reference" "J6" (at 106.68 72.39 0)
-      (effects (font (size 1.27 1.27)))
-    )
-    (property "Value" "Conn_01x16_P2.54MM_HeaderHoles" (at 109.22 92.71 90)
-      (effects (font (size 1.27 1.27)))
-    )
-    (property "Footprint" "Janelia:PinHeader_1x16_P2.54mm_Vertical_Holes" (at 107.95 92.71 0)
-      (effects (font (size 1.27 1.27)) hide)
-    )
-    (property "Datasheet" "~" (at 107.95 92.71 0)
-      (effects (font (size 1.27 1.27)) hide)
-    )
-    (pin "2")
-    (pin "16")
-    (pin "15")
-    (pin "4")
-    (pin "5")
-    (pin "12")
-    (pin "7")
-    (pin "8")
-    (pin "9")
-    (pin "14")
-    (pin "3")
-    (pin "10")
-    (pin "6")
-    (pin "13")
-    (pin "11")
-    (pin "1")
-    (instances
-      (project "pico-hat-stepper"
-        (path "/df2b2e89-e055-4140-95de-f1df723db034/69dff8eb-dcc1-4f17-9e1d-cf8103035e92"
-          (reference "J6") (unit 1)
-        )
-      )
-    )
-  )
-  (symbol (lib_id "Janelia:Conn_01x12_P2.54MM_HeaderHoles") (at 162.56 88.9 0) (unit 1)
-    (in_bom no) (on_board yes) (dnp no)
-    (property "Reference" "J7" (at 161.29 73.66 0)
-      (effects (font (size 1.27 1.27)))
-    )
-    (property "Value" "Conn_01x12_P2.54MM_HeaderHoles" (at 163.83 88.9 90)
-      (effects (font (size 1.27 1.27)))
-    )
-    (property "Footprint" "Janelia:PinHeader_1x12_P2.54mm_Vertical_Holes" (at 162.56 88.9 0)
-      (effects (font (size 1.27 1.27)) hide)
-    )
-    (property "Datasheet" "~" (at 162.56 88.9 0)
-      (effects (font (size 1.27 1.27)) hide)
-    )
-    (pin "9")
-    (pin "8")
-    (pin "7")
-    (pin "6")
-    (pin "1")
-    (pin "5")
-    (pin "3")
-    (pin "2")
-    (pin "12")
-    (pin "11")
-    (pin "10")
-    (pin "4")
-    (instances
-      (project "pico-hat-stepper"
-        (path "/df2b2e89-e055-4140-95de-f1df723db034/69dff8eb-dcc1-4f17-9e1d-cf8103035e92"
-          (reference "J7") (unit 1)
-        )
-      )
-    )
-  )
 )
