File: stepper-controller/assembly.kicad_sch (KiCad schematic)
At the start: 8 parts

Commit message: pico-hat-stepper -> stepper-controller
Other:
- title: pico-hat-stepper -> stepper-controller
Changed lines of the file:
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@@
   (paper "A4")
   (title_block
-    (title "pico-hat-stepper")
+    (title "stepper-controller")
     (date "2024-04-16")
     (rev "1.0")
@@
     (pin "1")
     (instances
-      (project "pico-hat-stepper"
+      (project "stepper-controller"
         (path "/df2b2e89-e055-4140-95de-f1df723db034/0ec4fe58-7f94-4826-b0e2-2bc8f3ffe81e"
           (reference "H1") (unit 1)
@@
     )
     (instances
-      (project "pico-hat-stepper"
+      (project "stepper-controller"
         (path "/df2b2e89-e055-4140-95de-f1df723db034/0ec4fe58-7f94-4826-b0e2-2bc8f3ffe81e"
           (reference "FID2") (unit 1)
@@
     (pin "1")
     (instances
-      (project "pico-hat-stepper"
+      (project "stepper-controller"
         (path "/df2b2e89-e055-4140-95de-f1df723db034/0ec4fe58-7f94-4826-b0e2-2bc8f3ffe81e"
           (reference "H3") (unit 1)
@@
     )
     (instances
-      (project "pico-hat-stepper"
+      (project "stepper-controller"
         (path "/df2b2e89-e055-4140-95de-f1df723db034/0ec4fe58-7f94-4826-b0e2-2bc8f3ffe81e"
           (reference "FID4") (unit 1)
@@
     )
     (instances
-      (project "pico-hat-stepper"
+      (project "stepper-controller"
         (path "/df2b2e89-e055-4140-95de-f1df723db034/0ec4fe58-7f94-4826-b0e2-2bc8f3ffe81e"
           (reference "FID1") (unit 1)
@@
     (pin "1")
     (instances
-      (project "pico-hat-stepper"
+      (project "stepper-controller"
         (path "/df2b2e89-e055-4140-95de-f1df723db034/0ec4fe58-7f94-4826-b0e2-2bc8f3ffe81e"
           (reference "H4") (unit 1)
@@
     (pin "1")
     (instances
-      (project "pico-hat-stepper"
+      (project "stepper-controller"
         (path "/df2b2e89-e055-4140-95de-f1df723db034/0ec4fe58-7f94-4826-b0e2-2bc8f3ffe81e"
           (reference "H2") (unit 1)
@@
     )
     (instances
-      (project "pico-hat-stepper"
+      (project "stepper-controller"
         (path "/df2b2e89-e055-4140-95de-f1df723db034/0ec4fe58-7f94-4826-b0e2-2bc8f3ffe81e"
           (reference "FID3") (unit 1)

Commit message: Add pico
Parts:
- removed H1, H2, H3, H4: MOUNTING_HOLE_2.5, Janelia:MOUNTING_HOLE_2.5, symbol Janelia:MOUNTING_HOLE_2.5
- added H1, H2, H3, H4: MountingHole_M3_Pad, Janelia:MountingHole_3.2mm_M3_Pad, symbol Janelia:MountingHole_M3_Pad
Connections:
- net GND: now also H1.1, H2.1, H3.1, H4.1
Changed lines of the file:
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@@
     (company "Howard Hughes Medical Institute")
   )
-  (wire (pts (xy 160.02 99.06) (xy 160.02 101.6))
+  (wire (pts (xy 149.86 138.43) (xy 149.86 140.97))
     (stroke (width 0) (type default))
   )
-  (wire (pts (xy 119.38 99.06) (xy 119.38 101.6))
+  (wire (pts (xy 149.86 110.49) (xy 149.86 113.03))
     (stroke (width 0) (type default))
   )
-  (wire (pts (xy 76.2 95.25) (xy 78.74 95.25))
+  (wire (pts (xy 149.86 96.52) (xy 149.86 99.06))
     (stroke (width 0) (type default))
   )
-  (wire (pts (xy 139.7 99.06) (xy 139.7 101.6))
+  (wire (pts (xy 111.76 91.44) (xy 114.3 91.44))
     (stroke (width 0) (type default))
   )
-  (wire (pts (xy 180.34 99.06) (xy 180.34 101.6))
+  (wire (pts (xy 149.86 124.46) (xy 149.86 127))
     (stroke (width 0) (type default))
   )
-  (label "GND" (at 119.38 101.6 270) (fields_autoplaced)
+  (label "GND" (at 149.86 113.03 270) (fields_autoplaced)
     (effects (font (size 1.27 1.27)) (justify right bottom))
   )
-  (label "GND" (at 78.74 95.25 0) (fields_autoplaced)
+  (label "GND" (at 149.86 99.06 270) (fields_autoplaced)
+    (effects (font (size 1.27 1.27)) (justify right bottom))
+  )
+  (label "GND" (at 114.3 91.44 0) (fields_autoplaced)
     (effects (font (size 1.27 1.27)) (justify left bottom))
   )
-  (label "GND" (at 160.02 101.6 270) (fields_autoplaced)
+  (label "GND" (at 149.86 140.97 270) (fields_autoplaced)
     (effects (font (size 1.27 1.27)) (justify right bottom))
   )
-  (label "GND" (at 180.34 101.6 270) (fields_autoplaced)
+  (label "GND" (at 149.86 127 270) (fields_autoplaced)
     (effects (font (size 1.27 1.27)) (justify right bottom))
   )
-  (label "GND" (at 139.7 101.6 270) (fields_autoplaced)
-    (effects (font (size 1.27 1.27)) (justify right bottom))
-  )
-  (hierarchical_label "GND" (shape passive) (at 76.2 95.25 180) (fields_autoplaced)
+  (hierarchical_label "GND" (shape passive) (at 111.76 91.44 180) (fields_autoplaced)
     (effects (font (size 1.27 1.27)) (justify right))
   )
-  (symbol (lib_id "Janelia:MOUNTING_HOLE_2.5") (at 119.38 99.06 0) (unit 1)
+  (symbol (lib_id "Janelia:MountingHole_M3_Pad") (at 149.86 93.98 0) (unit 1)
     (in_bom no) (on_board yes) (dnp no) (fields_autoplaced)
-    (property "Reference" "H1" (at 121.92 95.758 0)
+    (property "Reference" "H1" (at 152.4 91.44 0)
       (effects (font (size 1.27 1.27)) (justify left))
     )
-    (property "Value" "MOUNTING_HOLE_2.5" (at 119.38 106.68 0) (do_not_autoplace)
+    (property "Value" "MountingHole_M3_Pad" (at 152.4 93.98 0)
+      (effects (font (size 1.27 1.27)) (justify left))
+    )
+    (property "Footprint" "Janelia:MountingHole_3.2mm_M3_Pad" (at 149.86 93.98 0)
       (effects (font (size 1.27 1.27)) hide)
     )
-    (property "Footprint" "Janelia:MOUNTING_HOLE_2.5" (at 119.38 109.22 0) (do_not_autoplace)
-      (effects (font (size 1.27 1.27)) hide)
-    )
-    (property "Datasheet" "" (at 124.46 99.06 0)
-      (effects (font (size 1.27 1.27)) hide)
-    )
-    (property "Sim.Enable" "0" (at 119.38 99.06 0) (do_not_autoplace)
+    (property "Datasheet" "~" (at 149.86 93.98 0)
       (effects (font (size 1.27 1.27)) hide)
     )
@@
     )
   )
-  (symbol (lib_id "Janelia:MOUNTING_HOLE_2.5") (at 160.02 99.06 0) (unit 1)
+  (symbol (lib_id "Janelia:MountingHole_M3_Pad") (at 149.86 135.89 0) (unit 1)
     (in_bom no) (on_board yes) (dnp no) (fields_autoplaced)
-    (property "Reference" "H3" (at 162.56 95.758 0)
+    (property "Reference" "H4" (at 152.4 133.35 0)
       (effects (font (size 1.27 1.27)) (justify left))
     )
-    (property "Value" "MOUNTING_HOLE_2.5" (at 160.02 106.68 0) (do_not_autoplace)
+    (property "Value" "MountingHole_M3_Pad" (at 152.4 135.89 0)
+      (effects (font (size 1.27 1.27)) (justify left))
+    )
+    (property "Footprint" "Janelia:MountingHole_3.2mm_M3_Pad" (at 149.86 135.89 0)
       (effects (font (size 1.27 1.27)) hide)
     )
-    (property "Footprint" "Janelia:MOUNTING_HOLE_2.5" (at 160.02 109.22 0) (do_not_autoplace)
+    (property "Datasheet" "~" (at 149.86 135.89 0)
       (effects (font (size 1.27 1.27)) hide)
     )
-    (property "Datasheet" "" (at 165.1 99.06 0)
+    (pin "1")
+    (instances
+      (project "stepper-controller"
+        (path "/df2b2e89-e055-4140-95de-f1df723db034/0ec4fe58-7f94-4826-b0e2-2bc8f3ffe81e"
+          (reference "H4") (unit 1)
+        )
+      )
+    )
+  )
+  (symbol (lib_id "Janelia:MountingHole_M3_Pad") (at 149.86 121.92 0) (unit 1)
+    (in_bom no) (on_board yes) (dnp no) (fields_autoplaced)
+    (property "Reference" "H3" (at 152.4 119.38 0)
+      (effects (font (size 1.27 1.27)) (justify left))
+    )
+    (property "Value" "MountingHole_M3_Pad" (at 152.4 121.92 0)
+      (effects (font (size 1.27 1.27)) (justify left))
+    )
+    (property "Footprint" "Janelia:MountingHole_3.2mm_M3_Pad" (at 149.86 121.92 0)
       (effects (font (size 1.27 1.27)) hide)
     )
-    (property "Sim.Enable" "0" (at 160.02 99.06 0) (do_not_autoplace)
+    (property "Datasheet" "~" (at 149.86 121.92 0)
       (effects (font (size 1.27 1.27)) hide)
     )
@@
     )
   )
-  (symbol (lib_id "Janelia:MOUNTING_HOLE_2.5") (at 180.34 99.06 0) (unit 1)
+  (symbol (lib_id "Janelia:MountingHole_M3_Pad") (at 149.86 107.95 0) (unit 1)
     (in_bom no) (on_board yes) (dnp no) (fields_autoplaced)
-    (property "Reference" "H4" (at 182.88 95.758 0)
+    (property "Reference" "H2" (at 152.4 105.41 0)
       (effects (font (size 1.27 1.27)) (justify left))
     )
-    (property "Value" "MOUNTING_HOLE_2.5" (at 180.34 106.68 0) (do_not_autoplace)
+    (property "Value" "MountingHole_M3_Pad" (at 152.4 107.95 0)
+      (effects (font (size 1.27 1.27)) (justify left))
+    )
+    (property "Footprint" "Janelia:MountingHole_3.2mm_M3_Pad" (at 149.86 107.95 0)
       (effects (font (size 1.27 1.27)) hide)
     )
-    (property "Footprint" "Janelia:MOUNTING_HOLE_2.5" (at 180.34 109.22 0) (do_not_autoplace)
+    (property "Datasheet" "~" (at 149.86 107.95 0)
       (effects (font (size 1.27 1.27)) hide)
     )
-    (property "Datasheet" "" (at 185.42 99.06 0)
-      (effects (font (size 1.27 1.27)) hide)
-    )
-    (property "Sim.Enable" "0" (at 180.34 99.06 0) (do_not_autoplace)
-      (effects (font (size 1.27 1.27)) hide)
-    )
-    (pin "1")
-    (instances
-      (project "stepper-controller"
-        (path "/df2b2e89-e055-4140-95de-f1df723db034/0ec4fe58-7f94-4826-b0e2-2bc8f3ffe81e"
-          (reference "H4") (unit 1)
-        )
-      )
-    )
-  )
-  (symbol (lib_id "Janelia:MOUNTING_HOLE_2.5") (at 139.7 99.06 0) (unit 1)
-    (in_bom no) (on_board yes) (dnp no) (fields_autoplaced)
-    (property "Reference" "H2" (at 142.24 95.758 0)
-      (effects (font (size 1.27 1.27)) (justify left))
-    )
-    (property "Value" "MOUNTING_HOLE_2.5" (at 139.7 106.68 0) (do_not_autoplace)
-      (effects (font (size 1.27 1.27)) hide)
-    )
-    (property "Footprint" "Janelia:MOUNTING_HOLE_2.5" (at 139.7 109.22 0) (do_not_autoplace)
-      (effects (font (size 1.27 1.27)) hide)
-    )
-    (property "Datasheet" "" (at 144.78 99.06 0)
-      (effects (font (size 1.27 1.27)) hide)
-    )
-    (property "Sim.Enable" "0" (at 139.7 99.06 0) (do_not_autoplace)
-      (effects (font (size 1.27 1.27)) hide)
-    )
