File: stepper-controller/mosfet.kicad_sch (KiCad schematic)
At the start: 2 parts, among them U4 BUK7D36-60EX

Commit message: pico-hat-stepper -> stepper-controller
Other:
- title: pico-hat-stepper -> stepper-controller
Changed lines of the file:
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@@
   (paper "A4")
   (title_block
-    (title "pico-hat-stepper")
+    (title "stepper-controller")
     (date "2024-04-16")
     (rev "1.0")
@@
     (pin "8")
     (instances
-      (project "pico-hat-stepper"
+      (project "stepper-controller"
         (path "/df2b2e89-e055-4140-95de-f1df723db034/039ac378-5273-4081-85bf-9eb26cb5ed57/166b4ba4-5822-49d8-b309-f52ce04f60b1"
           (reference "U4") (unit 1)
@@
     (pin "1")
     (instances
-      (project "pico-hat-stepper"
+      (project "stepper-controller"
         (path "/df2b2e89-e055-4140-95de-f1df723db034/039ac378-5273-4081-85bf-9eb26cb5ed57/166b4ba4-5822-49d8-b309-f52ce04f60b1"
           (reference "R10") (unit 1)

Commit message: Add pico
Parts:
- renumbered U4 to U6
Changed lines of the file:
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@@
   (symbol (lib_id "Janelia:BUK7D36-60EX") (at 147.32 80.01 0) (unit 1)
     (in_bom yes) (on_board yes) (dnp no) (fields_autoplaced)
-    (property "Reference" "U4" (at 151.13 80.01 0) (do_not_autoplace)
+    (property "Reference" "U6" (at 151.13 80.01 0) (do_not_autoplace)
       (effects (font (size 1.524 1.524)) (justify left))
     )
@@
       (project "stepper-controller"
         (path "/df2b2e89-e055-4140-95de-f1df723db034/039ac378-5273-4081-85bf-9eb26cb5ed57/166b4ba4-5822-49d8-b309-f52ce04f60b1"
-          (reference "U4") (unit 1)
+          (reference "U6") (unit 1)
         )
         (path "/df2b2e89-e055-4140-95de-f1df723db034/039ac378-5273-4081-85bf-9eb26cb5ed57/77ec754f-e73d-4b40-8cb6-04aa79ed075b"
-          (reference "U5") (unit 1)
+          (reference "U7") (unit 1)
         )
         (path "/df2b2e89-e055-4140-95de-f1df723db034/039ac378-5273-4081-85bf-9eb26cb5ed57/3a5be366-e07c-4cea-9d17-ab6873df58d0"
-          (reference "U6") (unit 1)
+          (reference "U8") (unit 1)
         )
         (path "/df2b2e89-e055-4140-95de-f1df723db034/039ac378-5273-4081-85bf-9eb26cb5ed57/015fc9e7-3ba8-423b-8c7a-1e6ac6af06ca"
-          (reference "U7") (unit 1)
+          (reference "U9") (unit 1)
         )
         (path "/df2b2e89-e055-4140-95de-f1df723db034/039ac378-5273-4081-85bf-9eb26cb5ed57/310c6d75-c755-45f6-91bd-c6a3e28c41c3"
-          (reference "U8") (unit 1)
+          (reference "U10") (unit 1)
         )
         (path "/df2b2e89-e055-4140-95de-f1df723db034/039ac378-5273-4081-85bf-9eb26cb5ed57/e5ac0a82-cfa0-413a-a1a3-5e88ae5fe4fa"
-          (reference "U9") (unit 1)
+          (reference "U11") (unit 1)
         )
         (path "/df2b2e89-e055-4140-95de-f1df723db034/039ac378-5273-4081-85bf-9eb26cb5ed57/33c1e78d-612d-4de4-b4ab-c1f2402fd86d"
-          (reference "U10") (unit 1)
+          (reference "U12") (unit 1)
         )
         (path "/df2b2e89-e055-4140-95de-f1df723db034/039ac378-5273-4081-85bf-9eb26cb5ed57/3cc889de-698d-4e8a-bf98-2840b1fad77e"
-          (reference "U11") (unit 1)
+          (reference "U13") (unit 1)
         )
       )
