File: stepper-controller/pico-hat.kicad_sch (KiCad schematic)
At the start: 0 parts

Commit message: pico-hat-stepper -> stepper-controller
Other:
- title: pico-hat-stepper -> stepper-controller
Changed lines of the file:
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@@
   (paper "A4")
   (title_block
-    (title "pico-hat-stepper")
+    (title "stepper-controller")
     (date "2024-04-16")
     (rev "1.0")

Commit message: Add pico
Parts:
- added D4: DIODE_SCHOTTKY_20V_1A, Janelia:DIOM3616X98N, symbol Janelia:DIODE_SCHOTTKY_20V_1A
- added J5: PICO_LOW_HEADER_SMD, Janelia:Pico_Low_PinHeader_Vertical_SMD_Pin1Right, symbol Janelia:PICO_LOW_HEADER_SMD
- added J6: PICO_HIGH_HEADER_SMD, Janelia:Pico_High_PinHeader_Vertical_SMD_Pin1Right, symbol Janelia:PICO_HIGH_HEADER_SMD
Connections:
- net DIAG0: now also J5.9 (I2C1-SDA/SPI0-SCK/GP6)
- net DIAG1: now also J5.10 (I2C1-SCL/SPI0-TX/GP7)
- net ENABLE_FAN: now also J5.12 (UART1-RX/I2C0-SCL/SPI1-CS/GP9)
- net ENABLE_VIO: now also J5.11 (UART1-TX/I2C0-SDA/SPI1-RX/GP8)
- net GND: now also J6.38 (GND)
- net MISO: now also J6.26 (I2C0-SDA/GP20)
- net MOSI: now also J6.25 (I2C1-SCL/SPI0-TX/GP19)
- net SCK: now also J6.24 (I2C1-SDA/SPI0-SCK/GP18)
- net ~{CS}: now also J5.14 (I2C1-SDA/SPI1-SCK/GP10)
- new net: D4.1 (K), J6.39 (VSYS)
- new net VSYS: D4.2 (A)
- no-connect marks 0 -> 30
