File: stepper-controller/power.kicad_sch (KiCad schematic)
At the start: 14 parts, among them J1 Conn_01x03_P2.54MM_HeaderHoles, J2 Conn_01x02_P1.5MM_Molex_Pico-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, J3 Conn_01x03_P2.54MM_HeaderHoles, J8 HEADER_01X03_JST_SUR_VERTICAL, Q1 MOSFET-N-CH, U1 3.3V_100MA

Commit message: pico-hat-stepper -> stepper-controller
Other:
- title: pico-hat-stepper -> stepper-controller
Changed lines of the file:
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@@
   (paper "A4")
   (title_block
-    (title "pico-hat-stepper")
+    (title "stepper-controller")
     (date "2024-04-16")
     (rev "1.0")
@@
     (pin "3")
     (instances
-      (project "pico-hat-stepper"
+      (project "stepper-controller"
         (path "/df2b2e89-e055-4140-95de-f1df723db034/c1dd8f61-494c-402f-8e59-08309c64fc3f"
           (reference "J8") (unit 1)
@@
     (pin "1")
     (instances
-      (project "pico-hat-stepper"
+      (project "stepper-controller"
         (path "/df2b2e89-e055-4140-95de-f1df723db034/c1dd8f61-494c-402f-8e59-08309c64fc3f"
           (reference "C20") (unit 1)
@@
     (pin "3")
     (instances
-      (project "pico-hat-stepper"
+      (project "stepper-controller"
         (path "/df2b2e89-e055-4140-95de-f1df723db034/c1dd8f61-494c-402f-8e59-08309c64fc3f"
           (reference "J3") (unit 1)
@@
     (pin "1")
     (instances
-      (project "pico-hat-stepper"
+      (project "stepper-controller"
         (path "/df2b2e89-e055-4140-95de-f1df723db034/c1dd8f61-494c-402f-8e59-08309c64fc3f"
           (reference "R18") (unit 1)
@@
     (pin "2")
     (instances
-      (project "pico-hat-stepper"
+      (project "stepper-controller"
         (path "/df2b2e89-e055-4140-95de-f1df723db034/c1dd8f61-494c-402f-8e59-08309c64fc3f"
           (reference "D2") (unit 1)
@@
     (pin "1")
     (instances
-      (project "pico-hat-stepper"
+      (project "stepper-controller"
         (path "/df2b2e89-e055-4140-95de-f1df723db034/c1dd8f61-494c-402f-8e59-08309c64fc3f"
           (reference "C2") (unit 1)
@@
     (pin "1")
     (instances
-      (project "pico-hat-stepper"
+      (project "stepper-controller"
         (path "/df2b2e89-e055-4140-95de-f1df723db034/c1dd8f61-494c-402f-8e59-08309c64fc3f"
           (reference "J2") (unit 1)
@@
     (pin "3")
     (instances
-      (project "pico-hat-stepper"
+      (project "stepper-controller"
         (path "/df2b2e89-e055-4140-95de-f1df723db034/c1dd8f61-494c-402f-8e59-08309c64fc3f"
           (reference "J1") (unit 1)
@@
     (pin "3")
     (instances
-      (project "pico-hat-stepper"
+      (project "stepper-controller"
         (path "/df2b2e89-e055-4140-95de-f1df723db034/c1dd8f61-494c-402f-8e59-08309c64fc3f"
           (reference "U1") (unit 1)
@@
     (pin "1")
     (instances
-      (project "pico-hat-stepper"
+      (project "stepper-controller"
         (path "/df2b2e89-e055-4140-95de-f1df723db034/c1dd8f61-494c-402f-8e59-08309c64fc3f"
           (reference "Q1") (unit 1)
@@
     (pin "2")
     (instances
-      (project "pico-hat-stepper"
+      (project "stepper-controller"
         (path "/df2b2e89-e055-4140-95de-f1df723db034/c1dd8f61-494c-402f-8e59-08309c64fc3f"
           (reference "R2") (unit 1)
@@
     (pin "2")
     (instances
-      (project "pico-hat-stepper"
+      (project "stepper-controller"
         (path "/df2b2e89-e055-4140-95de-f1df723db034/c1dd8f61-494c-402f-8e59-08309c64fc3f"
           (reference "C1") (unit 1)
@@
     (pin "2")
     (instances
-      (project "pico-hat-stepper"
+      (project "stepper-controller"
         (path "/df2b2e89-e055-4140-95de-f1df723db034/c1dd8f61-494c-402f-8e59-08309c64fc3f"
           (reference "D1") (unit 1)
@@
     (pin "1")
     (instances
-      (project "pico-hat-stepper"
+      (project "stepper-controller"
         (path "/df2b2e89-e055-4140-95de-f1df723db034/c1dd8f61-494c-402f-8e59-08309c64fc3f"
           (reference "R1") (unit 1)

Commit message: Add pico
Parts:
- removed C1: 10uF_100V, Janelia:C_1210_3225Metric, symbol Janelia:C_10uF_100V_1210
- removed C20: 10uF_6.3V, Janelia:C_0402_1005Metric, symbol Janelia:C_10uF_6.3V_0402
- removed J1, J3: Conn_01x03_P2.54MM_HeaderHoles, Janelia:PinHeader_1x03_P2.54mm_Vertical_Holes, symbol Janelia:Conn_01x03_P2.54MM_HeaderHoles
- removed Q1: MOSFET-N-CH, Janelia:XFDFN-3, symbol Janelia:MOSFET-N-CH-EN-CSD17483F4
- removed R18: 15, Janelia:R_0402_1005Metric, symbol Janelia:R_15_0.1W_0402
- added C1, C2, C3: 1uF_100V, Janelia:C_0805_2012Metric, symbol Janelia:C_1uF_100V_0805
- added C4, C6: 10uF_6.3V, Janelia:C_0402_1005Metric, symbol Janelia:C_10uF_6.3V_0402
- added U1, U3: 3.3V_100MA, Janelia:DRB0008B, symbol Janelia:Regulator_Linear_3.3V_100MA_60Vin
- renumbered C2 to C5, J2 to J1, J8 to J2, U1 to U2
Connections:
- net VFAN- is gone; now on net GND: J2.3 (Pin_3)
- net ENABLE_FAN: now also U3.5 (EN)
- net GND: now also C1.2, C2.2, C3.2, C4.2, C6.2, U1.4 (GND), U1.9 (PAD), U3.4 (GND), U3.9 (PAD)
- net VM: now also C1.1, C2.1, C3.1, U1.5 (EN), U1.8 (IN), U3.8 (IN)
- net VFAN+ renamed VFAN
- net VFAN: now also C6.1, U3.1 (OUT)
- new net VSYS: C4.1, U1.1 (OUT)
- no-connect marks 3 -> 7
Other:
- moved on the sheet: C5, D1, D2, J1, J2, R1, R2, U2
