File: stepper-controller/stepper-controller.kicad_pcb (KiCad board)
At the start: 2 copper layers, 72 x 22.9 mm, 40 parts, among them J1 Conn_01x03_P2.54MM_HeaderHoles, J2 Conn_01x02_P1.5MM_Molex_Pico-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, J3 Conn_01x03_P2.54MM_HeaderHoles, J4 Conn_01x04_P1.5MM_Molex_Pico-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, J5 Conn_01x02_P1.5MM_Molex_Pico-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, J6 Conn_01x16_P2.54MM_HeaderHoles, J7 Conn_01x12_P2.54MM_HeaderHoles, U1 TMC5160A-WA, U10 3.3V_100MA, U11 MAX6816, U2 BUK7D36-60EX, U3 BUK7D36-60EX, U4 BUK7D36-60EX, U5 BUK7D36-60EX, U6 BUK7D36-60EX, U7 BUK7D36-60EX, U8 BUK7D36-60EX, U9 BUK7D36-60EX, X1 16MHz

Commit message: Add pico
Parts:
- removed J7: Conn_01x12_P2.54MM_HeaderHoles, Janelia:PinHeader_1x12_P2.54mm_Vertical_Holes
- added C10: 0.1uF_100V, Janelia:C_0402_1005Metric, F.Cu at (140.7, 139.8)
- added C11: 0.1uF_100V, Janelia:C_0402_1005Metric, F.Cu at (140.7, 141.8)
- added C12: 0.47uF_35V, Janelia:C_0402_1005Metric, F.Cu at (140.7, 143.8)
- added C13: 0.22uF_25V, Janelia:C_0402_1005Metric, F.Cu at (143.6, 137.9)
- added C14: 0.22uF_25V, Janelia:C_0402_1005Metric, F.Cu at (143.6, 139.8)
- added C15: 0.22uF_25V, Janelia:C_0402_1005Metric, F.Cu at (143.6, 141.8)
- added C16: 2.2uF_35V, Janelia:C_0402_1005Metric, F.Cu at (143.6, 143.8)
- added C17: 0.22uF_25V, Janelia:C_0402_1005Metric, F.Cu at (155.3, 138.4)
- added C18: 2.2uF_35V, Janelia:C_0402_1005Metric, F.Cu at (155.3, 141.4)
- added C19: 0.1uF_100V, Janelia:C_0402_1005Metric, F.Cu at (145.1, 129.3)
- added C20: 0.1uF_100V, Janelia:C_0402_1005Metric, F.Cu at (164.1, 129.7)
- added C21: 2.2uF_100V, Janelia:C_0805_2012Metric, F.Cu at (48.0, 66.6)
- added C22: 2.2uF_100V, Janelia:C_0805_2012Metric, F.Cu at (48.0, 69.6)
- added C23: 220uF_63V, Janelia:CP_Elec_EEEFK1J221AV, F.Cu at (54.5, 57.5)
- added C5: 10uF_6.3V, Janelia:C_0402_1005Metric, F.Cu at (137.8, 137.9)
- added C6: 10uF_6.3V, Janelia:C_0402_1005Metric, F.Cu at (137.8, 139.8)
- added C7: 0.1uF_100V, Janelia:C_0402_1005Metric, F.Cu at (137.8, 141.8)
- added C8: 22nF_100V, Janelia:C_0603_1608Metric, F.Cu at (137.8, 143.8)
- added C9: 0.1uF_100V, Janelia:C_0402_1005Metric, F.Cu at (140.7, 137.9)
- added D2: LED_GRN, Janelia:LED_0402_1005Metric, F.Cu at (161.2, 127.7)
- added D3: Diode_SMAJ51A, Janelia:D_SMA, F.Cu at (149.1, 139.2)
- added D4: DIODE_SCHOTTKY_20V_1A, Janelia:DIOM3616X98N, F.Cu at (40.6, 51.6)
- added R10: 15, Janelia:R_0402_1005Metric, F.Cu at (165.9, 133.6)
- added R11: 15, Janelia:R_0402_1005Metric, F.Cu at (165.9, 141.6)
- added R12: 15, Janelia:R_0402_1005Metric, F.Cu at (161.0, 141.6)
- added R13: 15, Janelia:R_0402_1005Metric, F.Cu at (161.0, 133.6)
- added R14: 15, Janelia:R_0402_1005Metric, F.Cu at (161.0, 137.6)
- added R15: 15, Janelia:R_0402_1005Metric, F.Cu at (165.9, 145.6)
- added R16: 15, Janelia:R_0402_1005Metric, F.Cu at (165.9, 137.6)
- added R17: 15, Janelia:R_0402_1005Metric, F.Cu at (161.0, 145.6)
- added R9: 0.15, Janelia:R_1206_3216Metric, F.Cu at (147.8, 143.1)
- added U12: BUK7D36-60EX, Janelia:BUK7D3660EX_NEX, F.Cu at (48.0, 75.0)
- added U13: BUK7D36-60EX, Janelia:BUK7D3660EX_NEX, F.Cu at (54.3, 75.0)
- C1, C2: value 100uF_63V -> 1uF_100V; footprint Janelia:CP_Elec_10x10.5 -> Janelia:C_0805_2012Metric
- C3: value 10uF_100V -> 1uF_100V; footprint Janelia:C_1210_3225Metric -> Janelia:C_0805_2012Metric
- D1: value Diode_SMAJ51A -> LED_RED; footprint Janelia:D_SMA -> Janelia:LED_0402_1005Metric
- H1, H2, H3, H4: value MOUNTING_HOLE_2.5 -> MountingHole_M3_Pad; footprint Janelia:MOUNTING_HOLE_2.5 -> Janelia:MountingHole_3.2mm_M3_Pad
- J1: value Conn_01x03_P2.54MM_HeaderHoles -> Conn_01x02_P1.5MM_Molex_Pico-SPOX-87438_Horizontal; footprint Janelia:PinHeader_1x03_P2.54mm_Vertical_Holes -> Janelia:Molex_Pico-SPOX-87438_1x02-P1.5MM_Horizontal
- J2: value Conn_01x02_P1.5MM_Molex_Pico-SPOX-87438_Horizontal -> HEADER_01X03_JST_SUR_VERTICAL; footprint Janelia:Molex_Pico-SPOX-87438_1x02-P1.5MM_Horizontal -> Janelia:JST_SUR_BM03B-SURS-TF_1x03-1MP_P0.80mm_Vertical
- J3: value Conn_01x03_P2.54MM_HeaderHoles -> Conn_01x02_P1.5MM_Molex_Pico-SPOX_Horizontal; footprint Janelia:PinHeader_1x03_P2.54mm_Vertical_Holes -> Janelia:Molex_Pico-Clasp-501568_1x02_P1MM_Horizontal
- J5: value Conn_01x02_P1.5MM_Molex_Pico-SPOX_Horizontal -> PICO_LOW_HEADER_SMD; footprint Janelia:Molex_Pico-Clasp-501568_1x02_P1MM_Horizontal -> Janelia:Pico_Low_PinHeader_Vertical_SMD_Pin1Right; moved to B.Cu
- J6: value Conn_01x16_P2.54MM_HeaderHoles -> PICO_HIGH_HEADER_SMD; footprint Janelia:PinHeader_1x16_P2.54mm_Vertical_Holes -> Janelia:Pico_High_PinHeader_Vertical_SMD_Pin1Right; moved to B.Cu
- R2: value 15 -> 64.9
- R3, R4, R7, R8: value 15 -> 47
- R5: value 15 -> 0.15; footprint Janelia:R_0402_1005Metric -> Janelia:R_1206_3216Metric
- R6: value 15 -> 2.2
- U1: value TMC5160A-WA -> 3.3V_100MA; footprint Janelia:21-100593_ADI -> Janelia:DRB0008B
- U10: value 3.3V_100MA -> BUK7D36-60EX; footprint Janelia:DRB0008B -> Janelia:BUK7D3660EX_NEX
- U11: value MAX6816 -> BUK7D36-60EX; footprint Janelia:SOT192P237X122-4N -> Janelia:BUK7D3660EX_NEX
- U2, U3: value BUK7D36-60EX -> 3.3V_100MA; footprint Janelia:BUK7D3660EX_NEX -> Janelia:DRB0008B
- U4: value BUK7D36-60EX -> TMC5160A-WA; footprint Janelia:BUK7D3660EX_NEX -> Janelia:21-100593_ADI
- U5: value BUK7D36-60EX -> MAX6816; footprint Janelia:BUK7D3660EX_NEX -> Janelia:SOT192P237X122-4N
- moved H3 66.3 mm to (241.4, 106.6)
- moved R4 53.8 mm to (215.8, 33.2)
- moved R5 53.8 mm to (215.8, 41.0)
- moved C3 53.8 mm to (203.2, 32.3)
- moved C4 53.8 mm to (196.8, 41.2)
- moved U2 53.8 mm to (240.0, 32.3)
- moved R1 53.8 mm to (228.6, 45.0)
- moved R2 53.8 mm to (222.2, 45.0)
- moved R3 53.8 mm to (228.6, 33.2)
- moved R6 53.8 mm to (228.6, 41.0)
- moved R7 53.8 mm to (222.2, 33.2)
- moved R8 53.8 mm to (222.2, 41.0)
- moved U10 53.8 mm to (194.3, 29.7)
- moved U3 53.8 mm to (240.0, 38.6)
- moved U4 53.8 mm to (229.3, 30.4)
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Connections:
- C4 pad 1: /VIO -> /VSYS
- D1 pad 1: /VM -> /GND
- D1 pad 2: /GND -> Net-(D1-A)
- J1 pad 2: /GND -> /VM
- J2 pad 1: /GND -> /power/VFAN
- J2 pad 2: /VM -> unconnected-(J2-Pin_2-Pad2)
- J3 pad 1: /VM -> /GND
- J3 pad 2: /VM -> /driver-controller/REFL
- J4 pad 1: unconnected-(J4-Pin_1-Pad1) -> /driver-controller/BMB2
- J4 pad 2: unconnected-(J4-Pin_2-Pad2) -> /driver-controller/BMB1
- J4 pad 3: unconnected-(J4-Pin_3-Pad3) -> /driver-controller/BMA2
- J4 pad 4: unconnected-(J4-Pin_4-Pad4) -> /driver-controller/BMA1
- R2 pad 1: /driver-controller/mosfet2/GATE -> /VIO
- R2 pad 2: Net-(U3-G) -> Net-(D2-A)
- R3 pad 1: /driver-controller/mosfet4/GATE -> /driver-controller/SRAH
- R3 pad 2: Net-(U4-G) -> /driver-controller/SRA
- R4 pad 1: /driver-controller/mosfet3/GATE -> /driver-controller/SRAL
- R4 pad 2: Net-(U5-G) -> /GND
- R5 pad 1: /driver-controller/mosfet5/GATE -> /driver-controller/SRA
- R5 pad 2: Net-(U6-G) -> /GND
- R6 pad 1: /driver-controller/mosfet6/GATE -> /driver-controller/VCC
- R6 pad 2: Net-(U7-G) -> /driver-controller/5VOUT
- R7 pad 1: /driver-controller/mosfet7/GATE -> /driver-controller/SRBH
- R7 pad 2: Net-(U8-G) -> /driver-controller/SRB
- R8 pad 1: /driver-controller/mosfet8/GATE -> /driver-controller/SRBL
- R8 pad 2: Net-(U9-G) -> /GND
- U1 pad 1: unconnected-(U1-BMB1-Pad1) -> /VSYS
- U1 pad 2: unconnected-(U1-HB1-Pad2) -> (no net)
- U1 pad 4: unconnected-(U1-12VOUT-Pad4) -> /GND
- U1 pad 5: unconnected-(U1-VSA-Pad5) -> /VM
- U1 pad 6: unconnected-(U1-5VOUT-Pad6) -> (no net)
- U1 pad 7: /GND -> unconnected-(U1-DELAY-Pad7)
- U1 pad 8: unconnected-(U1-SRAL-Pad8) -> /VM
- U1 pad 9: unconnected-(U1-SRAH-Pad9) -> /GND
- U10 pad 1: /VIO -> /VM
- U10 pad 2: (no net) -> /VM
- U10 pad 3: unconnected-(U10-PG-Pad3) -> Net-(U10-G)
- U10 pad 4: /GND -> /driver-controller/BMB2
- U10 pad 5: /power/ENABLE -> /VM
- U10 pad 6: (no net) -> /VM
- U10 pad 7: unconnected-(U10-DELAY-Pad7) -> /VM
- U10 pad 8: /VM -> /driver-controller/BMB2
- U11 pad 1: unconnected-(U11-GND-Pad1) -> /VM
- U11 pad 2: unconnected-(U11-IN-Pad2) -> /VM
- U11 pad 3: unconnected-(U11-OUT-Pad3) -> Net-(U11-G)
- U11 pad 4: unconnected-(U11-Vcc-Pad4) -> /driver-controller/BMB1
- U2 pad 1: /driver-controller/mosfet1/DRAIN -> /VIO
- U2 pad 2: /driver-controller/mosfet1/DRAIN -> (no net)
- U2 pad 3: Net-(U2-G) -> unconnected-(U2-PG-Pad3)
- U2 pad 4: /driver-controller/mosfet1/SOURCE -> /GND
- U2 pad 5: /driver-controller/mosfet1/DRAIN -> /ENABLE_VIO
- U2 pad 6: /driver-controller/mosfet1/DRAIN -> (no net)
- U2 pad 7: /driver-controller/mosfet1/DRAIN -> unconnected-(U2-DELAY-Pad7)
- U2 pad 8: /driver-controller/mosfet1/SOURCE -> /VM
- U3 pad 1: /driver-controller/mosfet2/DRAIN -> /power/VFAN
- U3 pad 2: /driver-controller/mosfet2/DRAIN -> (no net)
- U3 pad 3: Net-(U3-G) -> unconnected-(U3-PG-Pad3)
- U3 pad 4: /driver-controller/mosfet2/SOURCE -> /GND
- U3 pad 5: /driver-controller/mosfet2/DRAIN -> /ENABLE_FAN
- U3 pad 6: /driver-controller/mosfet2/DRAIN -> (no net)
- U3 pad 7: /driver-controller/mosfet2/DRAIN -> unconnected-(U3-DELAY-Pad7)
- U3 pad 8: /driver-controller/mosfet2/SOURCE -> /VM
- U4 pad 1: /driver-controller/mosfet4/DRAIN -> /driver-controller/BMB1
- U4 pad 2: /driver-controller/mosfet4/DRAIN -> /driver-controller/HB1
- U4 pad 3: Net-(U4-G) -> /driver-controller/CB1
- U4 pad 4: /driver-controller/mosfet4/SOURCE -> /driver-controller/12VOUT
- U4 pad 5: /driver-controller/mosfet4/DRAIN -> /VM
- U4 pad 6: /driver-controller/mosfet4/DRAIN -> /driver-controller/5VOUT
- U4 pad 7: /driver-controller/mosfet4/DRAIN -> /GND
- U4 pad 8: /driver-controller/mosfet4/SOURCE -> /driver-controller/SRAL
- U5 pad 1: /driver-controller/mosfet3/DRAIN -> /GND
- U5 pad 2: /driver-controller/mosfet3/DRAIN -> /driver-controller/REFL
- U5 pad 3: Net-(U5-G) -> /driver-controller/REFL_DEBOUNCED
- U5 pad 4: /driver-controller/mosfet3/SOURCE -> /VIO
- U6 pad 1: /driver-controller/mosfet5/DRAIN -> /VM
- U6 pad 2: /driver-controller/mosfet5/DRAIN -> /VM
- U6 pad 4: /driver-controller/mosfet5/SOURCE -> /driver-controller/BMA1
- U6 pad 5: /driver-controller/mosfet5/DRAIN -> /VM
- U6 pad 6: /driver-controller/mosfet5/DRAIN -> /VM
- U6 pad 7: /driver-controller/mosfet5/DRAIN -> /VM
- U6 pad 8: /driver-controller/mosfet5/SOURCE -> /driver-controller/BMA1
- U7 pad 1: /driver-controller/mosfet6/DRAIN -> /VM
- U7 pad 2: /driver-controller/mosfet6/DRAIN -> /VM
- U7 pad 4: /driver-controller/mosfet6/SOURCE -> /driver-controller/BMA2
- U7 pad 5: /driver-controller/mosfet6/DRAIN -> /VM
- U7 pad 6: /driver-controller/mosfet6/DRAIN -> /VM
- U7 pad 7: /driver-controller/mosfet6/DRAIN -> /VM
- U7 pad 8: /driver-controller/mosfet6/SOURCE -> /driver-controller/BMA2
- U8 pad 1: /driver-controller/mosfet7/DRAIN -> /driver-controller/BMA2
- U8 pad 2: /driver-controller/mosfet7/DRAIN -> /driver-controller/BMA2
- U8 pad 4: /driver-controller/mosfet7/SOURCE -> /driver-controller/SRA
- U8 pad 5: /driver-controller/mosfet7/DRAIN -> /driver-controller/BMA2
- U8 pad 6: /driver-controller/mosfet7/DRAIN -> /driver-controller/BMA2
- U8 pad 7: /driver-controller/mosfet7/DRAIN -> /driver-controller/BMA2
- U8 pad 8: /driver-controller/mosfet7/SOURCE -> /driver-controller/SRA
- U9 pad 1: /driver-controller/mosfet8/DRAIN -> /driver-controller/BMA1
- U9 pad 2: /driver-controller/mosfet8/DRAIN -> /driver-controller/BMA1
- U9 pad 4: /driver-controller/mosfet8/SOURCE -> /driver-controller/SRA
- U9 pad 5: /driver-controller/mosfet8/DRAIN -> /driver-controller/BMA1
- U9 pad 6: /driver-controller/mosfet8/DRAIN -> /driver-controller/BMA1
- U9 pad 7: /driver-controller/mosfet8/DRAIN -> /driver-controller/BMA1
- U9 pad 8: /driver-controller/mosfet8/SOURCE -> /driver-controller/SRA
