File: stepper-controller/stepper-controller.kicad_sch (KiCad schematic)
At the start: 0 parts

Commit message: pico-hat-stepper -> stepper-controller
Other:
- title: pico-hat-stepper -> stepper-controller
Changed lines of the file:
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@@
   (paper "A4")
   (title_block
-    (title "pico-hat-stepper")
+    (title "stepper-controller")
     (date "2024-04-16")
     (rev "1.0")
@@
     )
     (instances
-      (project "pico-hat-stepper"
+      (project "stepper-controller"
         (path "/df2b2e89-e055-4140-95de-f1df723db034" (page "4"))
       )
@@
     )
     (instances
-      (project "pico-hat-stepper"
+      (project "stepper-controller"
         (path "/df2b2e89-e055-4140-95de-f1df723db034" (page "2"))
       )
@@
     )
     (instances
-      (project "pico-hat-stepper"
+      (project "stepper-controller"
         (path "/df2b2e89-e055-4140-95de-f1df723db034" (page "13"))
       )
@@
     )
     (instances
-      (project "pico-hat-stepper"
+      (project "stepper-controller"
         (path "/df2b2e89-e055-4140-95de-f1df723db034" (page "3"))
       )

Commit message: Add pico
Other:
- sheet pico-hat ports: added VSYS; removed none
- sheet power ports: added VSYS; removed none
Changed lines of the file:
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@@
   (title_block
     (title "stepper-controller")
-    (date "2024-04-16")
+    (date "2024-04-17")
     (rev "1.0")
     (company "Howard Hughes Medical Institute")
@@
     (stroke (width 0) (type default))
   )
+  (wire (pts (xy 154.94 69.85) (xy 152.4 69.85))
+    (stroke (width 0) (type default))
+  )
   (wire (pts (xy 152.4 92.71) (xy 154.94 92.71))
     (stroke (width 0) (type default))
@@
     (stroke (width 0) (type default))
   )
-  (wire (pts (xy 154.94 69.85) (xy 152.4 69.85))
+  (wire (pts (xy 154.94 67.31) (xy 152.4 67.31))
     (stroke (width 0) (type default))
   )
@@
     (stroke (width 0) (type default))
   )
-  (wire (pts (xy 128.27 59.69) (xy 130.81 59.69))
+  (wire (pts (xy 128.27 55.88) (xy 130.81 55.88))
     (stroke (width 0) (type default))
   )
@@
     (stroke (width 0) (type default))
   )
+  (wire (pts (xy 128.27 90.17) (xy 130.81 90.17))
+    (stroke (width 0) (type default))
+  )
   (wire (pts (xy 152.4 95.25) (xy 154.94 95.25))
     (stroke (width 0) (type default))
@@
     (effects (font (size 1.27 1.27)) (justify right bottom))
   )
+  (label "VSYS" (at 154.94 69.85 0) (fields_autoplaced)
+    (effects (font (size 1.27 1.27)) (justify left bottom))
+  )
   (label "MOSI" (at 128.27 125.73 180) (fields_autoplaced)
     (effects (font (size 1.27 1.27)) (justify right bottom))
@@
     (effects (font (size 1.27 1.27)) (justify left bottom))
   )
+  (label "VSYS" (at 128.27 87.63 180) (fields_autoplaced)
+    (effects (font (size 1.27 1.27)) (justify right bottom))
+  )
   (label "VIO" (at 128.27 113.03 180) (fields_autoplaced)
     (effects (font (size 1.27 1.27)) (justify right bottom))
@@
     (effects (font (size 1.27 1.27)) (justify left bottom))
   )
-  (label "GND" (at 128.27 87.63 180) (fields_autoplaced)
-    (effects (font (size 1.27 1.27)) (justify right bottom))
-  )
-  (label "GND" (at 128.27 59.69 180) (fields_autoplaced)
+  (label "GND" (at 128.27 90.17 180) (fields_autoplaced)
+    (effects (font (size 1.27 1.27)) (justify right bottom))
+  )
+  (label "GND" (at 128.27 55.88 180) (fields_autoplaced)
     (effects (font (size 1.27 1.27)) (justify right bottom))
   )
@@
     (effects (font (size 1.27 1.27)) (justify right bottom))
   )
-  (label "VM" (at 154.94 69.85 0) (fields_autoplaced)
+  (label "VM" (at 154.94 67.31 0) (fields_autoplaced)
     (effects (font (size 1.27 1.27)) (justify left bottom))
   )
@@
     )
   )
-  (sheet (at 130.81 57.15) (size 21.59 5.08) (fields_autoplaced)
-    (stroke (width 0.1524) (type solid))
-    (fill (color 0 0 0 0.0000))
-    (property "Sheetname" "assembly" (at 130.81 56.4384 0)
-      (effects (font (size 1.27 1.27)) (justify left bottom))
-    )
-    (property "Sheetfile" "assembly.kicad_sch" (at 130.81 62.8146 0)
-      (effects (font (size 1.27 1.27)) (justify left top))
-    )
-    (pin "GND" passive (at 130.81 59.69 180)
+  (sheet (at 130.81 53.34) (size 21.59 5.08) (fields_autoplaced)
+    (stroke (width 0.1524) (type solid))
+    (fill (color 0 0 0 0.0000))
+    (property "Sheetname" "assembly" (at 130.81 52.6284 0)
+      (effects (font (size 1.27 1.27)) (justify left bottom))
+    )
+    (property "Sheetfile" "assembly.kicad_sch" (at 130.81 59.0046 0)
+      (effects (font (size 1.27 1.27)) (justify left top))
+    )
+    (pin "GND" passive (at 130.81 55.88 180)
       (effects (font (size 1.27 1.27)) (justify left))
     )
@@
       (effects (font (size 1.27 1.27)) (justify left top))
     )
-    (pin "GND" passive (at 130.81 87.63 180)
+    (pin "GND" passive (at 130.81 90.17 180)
       (effects (font (size 1.27 1.27)) (justify left))
     )
@@
     (pin "ENABLE_FAN" output (at 152.4 97.79 0)
       (effects (font (size 1.27 1.27)) (justify right))
+    )
+    (pin "VSYS" passive (at 130.81 87.63 180)
+      (effects (font (size 1.27 1.27)) (justify left))
     )
     (instances
@@
     )
   )
-  (sheet (at 130.81 67.31) (size 21.59 10.16) (fields_autoplaced)
-    (stroke (width 0.1524) (type solid))
-    (fill (color 0 0 0 0.0000))
-    (property "Sheetname" "power" (at 130.81 66.5984 0)
+  (sheet (at 130.81 64.77) (size 21.59 12.7) (fields_autoplaced)
+    (stroke (width 0.1524) (type solid))
+    (fill (color 0 0 0 0.0000))
+    (property "Sheetname" "power" (at 130.81 64.0584 0)
       (effects (font (size 1.27 1.27)) (justify left bottom))
     )
@@
       (effects (font (size 1.27 1.27)) (justify right))
     )
-    (pin "VM" passive (at 152.4 69.85 0)
+    (pin "VM" passive (at 152.4 67.31 0)
       (effects (font (size 1.27 1.27)) (justify right))
     )
@@
       (effects (font (size 1.27 1.27)) (justify left))
     )
-    (instances
+    (pin "VSYS" passive (at 152.4 69.85 0)
+      (effects (font (size 1.27 1.27)) (justify right))
+    )
+    (instances
