File: stepper-interface/driver-controller.kicad_sch (KiCad schematic)
At the start: 30 parts, among them J3 Conn_01x02_P1.5MM_Molex_Pico-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, J4 Conn_01x04_P1.5MM_Molex_Pico-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, U4 TMC5160A-WA, U5 MAX6816, X1 16MHz

Commit message: steppeer-controller -> stepper-interface
Other:
- title: stepper-controller -> stepper-interface
Changed lines of the file:
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@@
   (paper "A4")
   (title_block
-    (title "stepper-controller")
+    (title "stepper-interface")
     (date "2024-04-16")
     (rev "1.0")
@@
     (pin "2")
     (instances
-      (project "stepper-controller"
+      (project "stepper-interface"
         (path "/df2b2e89-e055-4140-95de-f1df723db034/039ac378-5273-4081-85bf-9eb26cb5ed57"
           (reference "C15") (unit 1)
@@
     (pin "2")
     (instances
-      (project "stepper-controller"
+      (project "stepper-interface"
         (path "/df2b2e89-e055-4140-95de-f1df723db034/039ac378-5273-4081-85bf-9eb26cb5ed57"
           (reference "R4") (unit 1)
@@
     (pin "1")
     (instances
-      (project "stepper-controller"
+      (project "stepper-interface"
         (path "/df2b2e89-e055-4140-95de-f1df723db034/039ac378-5273-4081-85bf-9eb26cb5ed57"
           (reference "C19") (unit 1)
@@
     (pin "2")
     (instances
-      (project "stepper-controller"
+      (project "stepper-interface"
         (path "/df2b2e89-e055-4140-95de-f1df723db034/039ac378-5273-4081-85bf-9eb26cb5ed57"
           (reference "C23") (unit 1)
@@
     (pin "2")
     (instances
-      (project "stepper-controller"
+      (project "stepper-interface"
         (path "/df2b2e89-e055-4140-95de-f1df723db034/039ac378-5273-4081-85bf-9eb26cb5ed57"
           (reference "C13") (unit 1)
@@
     (pin "1")
     (instances
-      (project "stepper-controller"
+      (project "stepper-interface"
         (path "/df2b2e89-e055-4140-95de-f1df723db034/039ac378-5273-4081-85bf-9eb26cb5ed57"
           (reference "C16") (unit 1)
@@
     (pin "3")
     (instances
-      (project "stepper-controller"
+      (project "stepper-interface"
         (path "/df2b2e89-e055-4140-95de-f1df723db034/039ac378-5273-4081-85bf-9eb26cb5ed57"
           (reference "J4") (unit 1)
@@
     (pin "2")
     (instances
-      (project "stepper-controller"
+      (project "stepper-interface"
         (path "/df2b2e89-e055-4140-95de-f1df723db034/039ac378-5273-4081-85bf-9eb26cb5ed57"
           (reference "U5") (unit 1)
@@
     (pin "1")
     (instances
-      (project "stepper-controller"
+      (project "stepper-interface"
         (path "/df2b2e89-e055-4140-95de-f1df723db034/039ac378-5273-4081-85bf-9eb26cb5ed57"
           (reference "C7") (unit 1)
@@
     (pin "2")
     (instances
-      (project "stepper-controller"
+      (project "stepper-interface"
         (path "/df2b2e89-e055-4140-95de-f1df723db034/039ac378-5273-4081-85bf-9eb26cb5ed57"
           (reference "C14") (unit 1)
@@
     (pin "1")
     (instances
-      (project "stepper-controller"
+      (project "stepper-interface"
         (path "/df2b2e89-e055-4140-95de-f1df723db034/039ac378-5273-4081-85bf-9eb26cb5ed57"
           (reference "C20") (unit 1)
@@
     (pin "18")
     (instances
-      (project "stepper-controller"
+      (project "stepper-interface"
         (path "/df2b2e89-e055-4140-95de-f1df723db034/039ac378-5273-4081-85bf-9eb26cb5ed57"
           (reference "U4") (unit 1)
@@
     (pin "2")
     (instances
-      (project "stepper-controller"
+      (project "stepper-interface"
         (path "/df2b2e89-e055-4140-95de-f1df723db034/039ac378-5273-4081-85bf-9eb26cb5ed57"
           (reference "C8") (unit 1)
@@
     (pin "1")
     (instances
-      (project "stepper-controller"
+      (project "stepper-interface"
         (path "/df2b2e89-e055-4140-95de-f1df723db034/039ac378-5273-4081-85bf-9eb26cb5ed57"
           (reference "C22") (unit 1)
@@
     (pin "2")
     (instances
-      (project "stepper-controller"
+      (project "stepper-interface"
         (path "/df2b2e89-e055-4140-95de-f1df723db034/039ac378-5273-4081-85bf-9eb26cb5ed57"
           (reference "R3") (unit 1)
@@
     (pin "1")
     (instances
-      (project "stepper-controller"
+      (project "stepper-interface"
         (path "/df2b2e89-e055-4140-95de-f1df723db034/039ac378-5273-4081-85bf-9eb26cb5ed57"
           (reference "R5") (unit 1)
@@
     (pin "1")
     (instances
-      (project "stepper-controller"
+      (project "stepper-interface"
         (path "/df2b2e89-e055-4140-95de-f1df723db034/039ac378-5273-4081-85bf-9eb26cb5ed57"
           (reference "#FLG03") (unit 1)
@@
     (pin "2")
     (instances
-      (project "stepper-controller"
+      (project "stepper-interface"
         (path "/df2b2e89-e055-4140-95de-f1df723db034/039ac378-5273-4081-85bf-9eb26cb5ed57"
           (reference "X1") (unit 1)
@@
     (pin "2")
     (instances
-      (project "stepper-controller"
+      (project "stepper-interface"
         (path "/df2b2e89-e055-4140-95de-f1df723db034/039ac378-5273-4081-85bf-9eb26cb5ed57"
           (reference "R7") (unit 1)
@@
     (pin "1")
     (instances
-      (project "stepper-controller"
+      (project "stepper-interface"
         (path "/df2b2e89-e055-4140-95de-f1df723db034/039ac378-5273-4081-85bf-9eb26cb5ed57"
           (reference "C12") (unit 1)
@@
     (pin "2")
     (instances
-      (project "stepper-controller"
+      (project "stepper-interface"
         (path "/df2b2e89-e055-4140-95de-f1df723db034/039ac378-5273-4081-85bf-9eb26cb5ed57"
           (reference "J3") (unit 1)
@@
     (pin "1")
     (instances
-      (project "stepper-controller"
+      (project "stepper-interface"
         (path "/df2b2e89-e055-4140-95de-f1df723db034/039ac378-5273-4081-85bf-9eb26cb5ed57"
           (reference "D3") (unit 1)
@@
     (pin "2")
     (instances
-      (project "stepper-controller"
+      (project "stepper-interface"
         (path "/df2b2e89-e055-4140-95de-f1df723db034/039ac378-5273-4081-85bf-9eb26cb5ed57"
           (reference "C17") (unit 1)
@@
     (pin "2")
     (instances
-      (project "stepper-controller"
+      (project "stepper-interface"
         (path "/df2b2e89-e055-4140-95de-f1df723db034/039ac378-5273-4081-85bf-9eb26cb5ed57"
           (reference "R8") (unit 1)
@@
     (pin "2")
     (instances
-      (project "stepper-controller"
+      (project "stepper-interface"
         (path "/df2b2e89-e055-4140-95de-f1df723db034/039ac378-5273-4081-85bf-9eb26cb5ed57"
           (reference "R6") (unit 1)
@@
     (pin "1")
     (instances
-      (project "stepper-controller"
+      (project "stepper-interface"
         (path "/df2b2e89-e055-4140-95de-f1df723db034/039ac378-5273-4081-85bf-9eb26cb5ed57"
           (reference "C10") (unit 1)
@@
     (pin "1")
     (instances
-      (project "stepper-controller"
+      (project "stepper-interface"
         (path "/df2b2e89-e055-4140-95de-f1df723db034/039ac378-5273-4081-85bf-9eb26cb5ed57"
           (reference "R9") (unit 1)
@@
     (pin "1")
     (instances
-      (project "stepper-controller"
+      (project "stepper-interface"
         (path "/df2b2e89-e055-4140-95de-f1df723db034/039ac378-5273-4081-85bf-9eb26cb5ed57"
           (reference "C18") (unit 1)
@@
     (pin "1")
     (instances
-      (project "stepper-controller"
+      (project "stepper-interface"
         (path "/df2b2e89-e055-4140-95de-f1df723db034/039ac378-5273-4081-85bf-9eb26cb5ed57"
           (reference "C21") (unit 1)
@@
     (pin "1")
     (instances
-      (project "stepper-controller"
+      (project "stepper-interface"
         (path "/df2b2e89-e055-4140-95de-f1df723db034/039ac378-5273-4081-85bf-9eb26cb5ed57"
           (reference "C9") (unit 1)
@@
     (pin "1")
     (instances
-      (project "stepper-controller"
+      (project "stepper-interface"
         (path "/df2b2e89-e055-4140-95de-f1df723db034/039ac378-5273-4081-85bf-9eb26cb5ed57"
           (reference "C11") (unit 1)
@@
     )
     (instances
-      (project "stepper-controller"
+      (project "stepper-interface"
         (path "/df2b2e89-e055-4140-95de-f1df723db034/039ac378-5273-4081-85bf-9eb26cb5ed57" (page "8"))
       )
@@
     )
     (instances
-      (project "stepper-controller"
+      (project "stepper-interface"
         (path "/df2b2e89-e055-4140-95de-f1df723db034/039ac378-5273-4081-85bf-9eb26cb5ed57" (page "5"))
       )
@@
     )
     (instances
-      (project "stepper-controller"
+      (project "stepper-interface"
         (path "/df2b2e89-e055-4140-95de-f1df723db034/039ac378-5273-4081-85bf-9eb26cb5ed57" (page "9"))
       )
@@
     )
     (instances
-      (project "stepper-controller"
+      (project "stepper-interface"
         (path "/df2b2e89-e055-4140-95de-f1df723db034/039ac378-5273-4081-85bf-9eb26cb5ed57" (page "11"))
       )
@@
     )
     (instances
-      (project "stepper-controller"
+      (project "stepper-interface"
         (path "/df2b2e89-e055-4140-95de-f1df723db034/039ac378-5273-4081-85bf-9eb26cb5ed57" (page "7"))
       )
@@
     )
     (instances
-      (project "stepper-controller"
+      (project "stepper-interface"
         (path "/df2b2e89-e055-4140-95de-f1df723db034/039ac378-5273-4081-85bf-9eb26cb5ed57" (page "12"))
       )
@@
     )
     (instances
-      (project "stepper-controller"
+      (project "stepper-interface"
         (path "/df2b2e89-e055-4140-95de-f1df723db034/039ac378-5273-4081-85bf-9eb26cb5ed57" (page "6"))
       )
@@
     )
     (instances
-      (project "stepper-controller"
+      (project "stepper-interface"
         (path "/df2b2e89-e055-4140-95de-f1df723db034/039ac378-5273-4081-85bf-9eb26cb5ed57" (page "10"))
       )
