File: stepper-interface/pico-hat.kicad_sch (KiCad schematic)
At the start: 3 parts, among them J5 PICO_LOW_HEADER_SMD, J6 PICO_HIGH_HEADER_SMD

Commit message: steppeer-controller -> stepper-interface
Other:
- title: stepper-controller -> stepper-interface
Changed lines of the file:
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@@
   (paper "A4")
   (title_block
-    (title "stepper-controller")
+    (title "stepper-interface")
     (date "2024-04-16")
     (rev "1.0")
@@
     (pin "3")
     (instances
-      (project "stepper-controller"
+      (project "stepper-interface"
         (path "/df2b2e89-e055-4140-95de-f1df723db034/69dff8eb-dcc1-4f17-9e1d-cf8103035e92"
           (reference "J5") (unit 1)
@@
     (pin "22")
     (instances
-      (project "stepper-controller"
+      (project "stepper-interface"
         (path "/df2b2e89-e055-4140-95de-f1df723db034/69dff8eb-dcc1-4f17-9e1d-cf8103035e92"
           (reference "J6") (unit 1)
@@
     (pin "1")
     (instances
-      (project "stepper-controller"
+      (project "stepper-interface"
         (path "/df2b2e89-e055-4140-95de-f1df723db034/69dff8eb-dcc1-4f17-9e1d-cf8103035e92"
           (reference "D4") (unit 1)
