File: stepper-interface/rp2040.kicad_sch (KiCad schematic)
At the start: 31 parts, among them J1301 Connector_USB_C_Receptacle, SW1301 Switch_Tactile_SPST-NO_SMT_Si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, U1301 Linear_3.3V_1A, U1302 MCU_RP2040, U1303 Memory_Flash_W25Q128JVZPIQ, Y1301 Crystal_12MHz

Commit message: First attempt at production files
Parts:
- C1301, C1302: Comment (none) -> 1 µF ±10% 25V Ceramic Capacitor X5R 0402 (1005 Metric)
- C1303, C1311: Comment (none) -> 1 µF ±10% 35V Ceramic Capacitor X5R 0402 (1005 Metric)
- C1304, C1305, C1306, C1307, C1308, C1309, C1310, C1312, C1313, C1314: Comment (none) -> 0.1 µF ±10% 100V Ceramic Capacitor X5R 0402 (1005 Metric)
- C1315, C1316: Comment (none) -> 15 pF ±5% 25V Ceramic Capacitor C0G, NP0 0402 (1005 Metric)
- D1301, D1302: Comment (none) -> Diode 40 V 2A Surface Mount 2-DSN (1.6x0.8), (0603)
- J1301: Comment (none) -> USB-C (USB TYPE-C) USB 3.2 Gen 2 (USB 3.1 Gen 2, Superspeed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
- R1301: Comment (none) -> 10 kOhms ±5% 0.063W, 1/16W Chip Resistor 0402 (1005 Metric)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
- R1302, R1303: Comment (none) -> 5.1 kOhms ±5% 0.1W, 1/10W Chip Resistor 0402 (1005 Metric) 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
- R1304, R1305: Comment (none) -> 27 Ohms ±5% 0.1W, 1/10W Chip Resistor 0402 (1005 Metric) Au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
- R1306, R1307: Comment (none) -> 1 kOhms ±1% 0.063W, 1/16W Chip Resistor 0402 (1005 Metric) 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
- SW1301: Comment (none) -> Tactile Switch SPST-NO Side Actuated Surface Mount, Right A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
- U1301: Comment (none) -> Linear Voltage Regulator IC Positive Fixed 1 Output 1A 8-SO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
- U1302: Comment (none) -> ARM® Cortex®-M0+ - Microcontroller IC 32-Bit Dual-Core 133M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
- U1303: Comment (none) -> FLASH - NOR Memory IC 128Mbit SPI - Quad I/O, QPI, DTR 133 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
- Y1301: Comment (none) -> 12 MHz ±30ppm Crystal 10pF 50 Ohms 4-SMD, No Lead
Changed lines of the file:
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@@
       (effects (font (size 1.524 1.524)) hide)
+    )
+    (property "Comment" "1 kOhms ±1% 0.063W, 1/16W Chip Resistor 0402 (1005 Metric) Moisture Resistant Thick Film" (at 256.54 116.84 0)
+      (effects (font (size 1.27 1.27)) hide)
     )
     (pin "1")
@@
       (effects (font (size 1.524 1.524)) hide)
     )
+    (property "Comment" "1 µF ±10% 35V Ceramic Capacitor X5R 0402 (1005 Metric)" (at 175.26 68.58 0)
+      (effects (font (size 1.27 1.27)) hide)
+    )
     (pin "2")
     (pin "1")
@@
       (effects (font (size 1.524 1.524)) hide)
     )
+    (property "Comment" "15 pF ±5% 25V Ceramic Capacitor C0G, NP0 0402 (1005 Metric)" (at 71.12 172.72 0)
+      (effects (font (size 1.27 1.27)) hide)
+    )
     (pin "2")
     (pin "1")
@@
       (effects (font (size 1.524 1.524)) hide)
     )
+    (property "Comment" "0.1 µF ±10% 100V Ceramic Capacitor X5R 0402 (1005 Metric)" (at 231.14 39.37 0)
+      (effects (font (size 1.27 1.27)) hide)
+    )
     (pin "2")
     (pin "1")
@@
       (effects (font (size 1.524 1.524)) hide)
     )
+    (property "Comment" "0.1 µF ±10% 100V Ceramic Capacitor X5R 0402 (1005 Metric)" (at 259.08 39.37 0)
+      (effects (font (size 1.27 1.27)) hide)
+    )
     (pin "2")
     (pin "1")
@@
     (property "Synopsis" "CAP CER 0.1UF 100V X5R" (at 210.82 58.42 0)
       (effects (font (size 1.524 1.524)) hide)
+    )
+    (property "Comment" "0.1 µF ±10% 100V Ceramic Capacitor X5R 0402 (1005 Metric)" (at 203.2 68.58 0)
+      (effects (font (size 1.27 1.27)) hide)
     )
     (pin "2")
@@
       (effects (font (size 1.27 1.27)) hide)
     )
+    (property "Comment" "Tactile Switch SPST-NO Side Actuated Surface Mount, Right Angle" (at 256.54 128.27 0)
+      (effects (font (size 1.27 1.27)) hide)
+    )
     (pin "4")
     (pin "3")
@@
       (effects (font (size 1.524 1.524)) hide)
     )
+    (property "Comment" "0.1 µF ±10% 100V Ceramic Capacitor X5R 0402 (1005 Metric)" (at 189.23 39.37 0)
+      (effects (font (size 1.27 1.27)) hide)
+    )
     (pin "2")
     (pin "1")
@@
     (property "Synopsis" "CAP CER 0.1UF 100V X5R" (at 224.79 29.21 0)
       (effects (font (size 1.524 1.524)) hide)
+    )
+    (property "Comment" "0.1 µF ±10% 100V Ceramic Capacitor X5R 0402 (1005 Metric)" (at 217.17 39.37 0)
+      (effects (font (size 1.27 1.27)) hide)
     )
     (pin "2")
@@
       (effects (font (size 1.27 1.27)) hide)
     )
+    (property "Comment" "Diode 40 V 2A Surface Mount 2-DSN (1.6x0.8), (0603)" (at 66.04 36.83 0)
+      (effects (font (size 1.27 1.27)) hide)
+    )
     (pin "2")
     (pin "1")
@@
     (property "Synopsis" "CAP CER 0.1UF 100V X5R" (at 231.14 104.14 0)
       (effects (font (size 1.524 1.524)) hide)
+    )
+    (property "Comment" "0.1 µF ±10% 100V Ceramic Capacitor X5R 0402 (1005 Metric)" (at 223.52 114.3 0)
+      (effects (font (size 1.27 1.27)) hide)
     )
     (pin "2")
@@
     )
     (property "Manufacturer Part Number" "GRT155R61E105KE01D" (at 90.17 39.37 0)
+      (effects (font (size 1.27 1.27)) hide)
+    )
+    (property "Comment" "1 µF ±10% 25V Ceramic Capacitor X5R 0402 (1005 Metric)" (at 90.17 39.37 0)
       (effects (font (size 1.27 1.27)) hide)
     )
@@
       (effects (font (size 1.524 1.524)) hide)
     )
+    (property "Comment" "5.1 kOhms ±5% 0.1W, 1/10W Chip Resistor 0402 (1005 Metric) Automotive AEC-Q200 Thick Film" (at 54.61 113.03 0)
+      (effects (font (size 1.27 1.27)) hide)
+    )
     (pin "1")
     (pin "2")
@@
       (effects (font (size 1.524 1.524)) hide)
     )
+    (property "Comment" "0.1 µF ±10% 100V Ceramic Capacitor X5R 0402 (1005 Metric)" (at 273.05 39.37 0)
+      (effects (font (size 1.27 1.27)) hide)
+    )
     (pin "2")
     (pin "1")
@@
       (effects (font (size 1.524 1.524)) hide)
     )
+    (property "Comment" "0.1 µF ±10% 100V Ceramic Capacitor X5R 0402 (1005 Metric)" (at 189.23 68.58 0)
+      (effects (font (size 1.27 1.27)) hide)
+    )
     (pin "2")
     (pin "1")
@@
     (property "Synopsis" "CAP CER 0.1UF 100V X5R" (at 210.82 29.21 0)
       (effects (font (size 1.524 1.524)) hide)
+    )
+    (property "Comment" "0.1 µF ±10% 100V Ceramic Capacitor X5R 0402 (1005 Metric)" (at 203.2 39.37 0)
+      (effects (font (size 1.27 1.27)) hide)
     )
     (pin "2")
@@
       (effects (font (size 1.524 1.524)) hide)
     )
+    (property "Comment" "5.1 kOhms ±5% 0.1W, 1/10W Chip Resistor 0402 (1005 Metric) Automotive AEC-Q200 Thick Film" (at 60.96 113.03 0)
+      (effects (font (size 1.27 1.27)) hide)
+    )
     (pin "1")
     (pin "2")
@@
       (effects (font (size 1.27 1.27)) hide)
     )
+    (property "Comment" "1 µF ±10% 25V Ceramic Capacitor X5R 0402 (1005 Metric)" (at 143.51 39.37 0)
+      (effects (font (size 1.27 1.27)) hide)
+    )
     (pin "2")
     (pin "1")
@@
     (property "Synopsis" "CAP CER 0.1UF 100V X5R" (at 252.73 29.21 0)
       (effects (font (size 1.524 1.524)) hide)
+    )
+    (property "Comment" "0.1 µF ±10% 100V Ceramic Capacitor X5R 0402 (1005 Metric)" (at 245.11 39.37 0)
+      (effects (font (size 1.27 1.27)) hide)
     )
     (pin "2")
@@
     )
     (property "Vendor Part Number" "609-10152803-00011LFCT-ND" (at 31.75 100.33 0)
+      (effects (font (size 1.27 1.27)) hide)
+    )
+    (property "Comment" "USB-C (USB TYPE-C) USB 3.2 Gen 2 (USB 3.1 Gen 2, Superspeed + (USB 3.1)) Receptacle Connector 24 Position Surface Mount, Right Angle" (at 31.75 100.33 0)
       (effects (font (size 1.27 1.27)) hide)
     )
@@
       (effects (font (size 1.27 1.27)) hide)
     )
+    (property "Comment" "Diode 40 V 2A Surface Mount 2-DSN (1.6x0.8), (0603)" (at 66.04 43.18 0)
+      (effects (font (size 1.27 1.27)) hide)
+    )
     (pin "2")
     (pin "1")
@@
     )
     (property "Vendor Part Number" "296-24157-1-ND" (at 119.38 17.78 0)
+      (effects (font (size 1.27 1.27)) hide)
+    )
+    (property "Comment" "Linear Voltage Regulator IC Positive Fixed 1 Output 1A 8-SON (3x3)" (at 119.38 39.37 0)
       (effects (font (size 1.27 1.27)) hide)
     )
@@
     )
     (property "Synopsis" "IC FLASH 128MBIT SPI/QUAD" (at 233.68 142.24 0)
+      (effects (font (size 1.27 1.27)) hide)
+    )
+    (property "Comment" "FLASH - NOR Memory IC 128Mbit SPI - Quad I/O, QPI, DTR 133 MHz 8-WSON (6x5)" (at 233.68 142.24 0)
       (effects (font (size 1.27 1.27)) hide)
     )
@@
       (effects (font (size 1.524 1.524)) hide)
     )
+    (property "Comment" "27 Ohms ±5% 0.1W, 1/10W Chip Resistor 0402 (1005 Metric) Automotive AEC-Q200 Thick Film" (at 67.31 113.03 0)
+      (effects (font (size 1.27 1.27)) hide)
+    )
     (pin "2")
     (pin "1")
@@
     )
     (property "Synopsis" "IC MCU 32BIT EXT MEM" (at 121.92 120.65 0)
+      (effects (font (size 1.27 1.27)) hide)
+    )
+    (property "Comment" "ARM® Cortex®-M0+ - Microcontroller IC 32-Bit Dual-Core 133MHz External Program Memory 56-QFN (7x7)" (at 121.92 120.65 0)
       (effects (font (size 1.27 1.27)) hide)
     )
@@
       (effects (font (size 1.524 1.524)) hide)
     )
+    (property "Comment" "15 pF ±5% 25V Ceramic Capacitor C0G, NP0 0402 (1005 Metric)" (at 58.42 172.72 0)
+      (effects (font (size 1.27 1.27)) hide)
+    )
     (pin "2")
     (pin "1")
@@
     (property "Synopsis" "CAP CER 1UF 35V X5R" (at 182.88 29.21 0)
       (effects (font (size 1.524 1.524)) hide)
+    )
+    (property "Comment" "1 µF ±10% 35V Ceramic Capacitor X5R 0402 (1005 Metric)" (at 175.26 39.37 0)
+      (effects (font (size 1.27 1.27)) hide)
     )
     (pin "2")
@@
       (effects (font (size 1.524 1.524)) hide)
     )
+    (property "Comment" "1 kOhms ±1% 0.063W, 1/16W Chip Resistor 0402 (1005 Metric) Moisture Resistant Thick Film" (at 39.37 172.72 0)
+      (effects (font (size 1.27 1.27)) hide)
+    )
     (pin "1")
     (pin "2")
@@
       (effects (font (size 1.524 1.524)) hide)
     )
+    (property "Comment" "10 kOhms ±5% 0.063W, 1/16W Chip Resistor 0402 (1005 Metric) Moisture Resistant Thick Film" (at 256.54 111.76 0)
+      (effects (font (size 1.27 1.27)) hide)
+    )
     (pin "1")
     (pin "2")
@@
       (effects (font (size 1.524 1.524)) hide)
     )
+    (property "Comment" "27 Ohms ±5% 0.1W, 1/10W Chip Resistor 0402 (1005 Metric) Automotive AEC-Q200 Thick Film" (at 73.66 113.03 0)
+      (effects (font (size 1.27 1.27)) hide)
+    )
     (pin "2")
     (pin "1")
@@
       (effects (font (size 1.27 1.27)) hide)
     )
+    (property "Comment" "12 MHz ±30ppm Crystal 10pF 50 Ohms 4-SMD, No Lead" (at 39.37 157.48 0)
+      (effects (font (size 1.27 1.27)) hide)
+    )

Commit message: Update schematic fields
Parts:
- C1301, C1302: Comment 1 µF ±10% 25V Ceramic Capacitor X5R 0402 (1005 Metric) -> Murata Electronics GRT155R61E105KE01D 1 µF ±10% 25V Ceramic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; LCSC (none) -> C711085
- C1303, C1311: Comment 1 µF ±10% 35V Ceramic Capacitor X5R 0402 (1005 Metric) -> Samsung Electro-Mechanics CL05A105KL5NRNC 1 µF ±10% 35V Cer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; LCSC (none) -> C307413
- C1304, C1305, C1306, C1307, C1308, C1309, C1310, C1312, C1313, C1314: Comment 0.1 µF ±10% 100V Ceramic Capacitor X5R 0402 (1005 Metric) -> Murata Electronics GRM155R62A104KE14D 0.1 µF ±10% 100V Cera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; LCSC (none) -> C162178
- C1315, C1316: Comment 15 pF ±5% 25V Ceramic Capacitor C0G, NP0 0402 (1005 Metric) -> KEMET C0402C150J3GACAUTO 15 pF ±5% 25V Ceramic Capacitor C0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; LCSC (none) -> C3888936
- D1301, D1302: Comment Diode 40 V 2A Surface Mount 2-DSN (1.6x0.8), (0603) -> onsemi NSR20F40NXT5G Diode 40 V 2A Surface Mount 2-DSN (1.6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; LCSC (none) -> C153761
- J1301: Comment USB-C (USB TYPE-C) USB 3.2 Gen 2 (USB 3.1 Gen 2, Superspeed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 -> Amphenol ICC (FCI) 10152803-00011LF USB-C (USB TYPE-C) USB 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; LCSC (none) -> C5410523
- R1301: Comment 10 kOhms ±5% 0.063W, 1/16W Chip Resistor 0402 (1005 Metric)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 -> YAGEO RC0402JR-0710KL 10 kOhms ±5% 0.063W, 1/16W Chip Resis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; LCSC (none) -> C106234
- R1302, R1303: Comment 5.1 kOhms ±5% 0.1W, 1/10W Chip Resistor 0402 (1005 Metric) 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 -> Panasonic Electronic Components ERJ-2GEJ512X 5.1 kOhms ±5% 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
- R1304, R1305: Comment 27 Ohms ±5% 0.1W, 1/10W Chip Resistor 0402 (1005 Metric) Au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 -> Panasonic Electronic Components ERJ-2GEJ270X 27 Ohms ±5% 0.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
- R1306, R1307: Comment 1 kOhms ±1% 0.063W, 1/16W Chip Resistor 0402 (1005 Metric) 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 -> YAGEO RC0402FR-071KL 1 kOhms ±1% 0.063W, 1/16W Chip Resisto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; LCSC (none) -> C106235
- SW1301: Comment Tactile Switch SPST-NO Side Actuated Surface Mount, Right A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 -> Würth Elektronik 436333045822 Tactile Switch SPST-NO Side A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; LCSC (none) -> C7185056
- U1301: Comment Linear Voltage Regulator IC Positive Fixed 1 Output 1A 8-SO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 -> Texas Instruments TPS73733QDRBRQ1 Linear Voltage Regulator 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; LCSC (none) -> C523768
- U1302: Comment ARM® Cortex®-M0+ - Microcontroller IC 32-Bit Dual-Core 133M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 -> Raspberry Pi SC0914(13) ARM Cortex-M0+ - Microcontroller IC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; LCSC (none) -> C3227924
- U1303: Comment FLASH - NOR Memory IC 128Mbit SPI - Quad I/O, QPI, DTR 133 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 -> Winbond Electronics W25Q128JVPIQ FLASH - NOR Memory IC 128M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; LCSC (none) -> C190862
- Y1301: Comment 12 MHz ±30ppm Crystal 10pF 50 Ohms 4-SMD, No Lead -> Abracon LLC ABM8-272-T3 12 MHz ±30ppm Crystal 10pF 50 Ohms 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; LCSC (none) -> C20625731

Commit message: Update LCSC part numbers
Parts:
- R1302, R1303: LCSC (none) -> C413002
- R1304, R1305: LCSC (none) -> C278580
Changed lines of the file:
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@@
   (title_block
     (title "stepper-interface")
-    (date "2024-05-08")
+    (date "2024-05-09")
     (rev "1.0")
     (company "Howard Hughes Medical Institute")
@@
       (effects (font (size 1.27 1.27)) hide)
     )
-    (property "LCSC" "" (at 54.61 113.03 0)
+    (property "LCSC" "C413002" (at 54.61 113.03 0)
       (effects (font (size 1.27 1.27)) hide)
     )
@@
       (effects (font (size 1.27 1.27)) hide)
     )
-    (property "LCSC" "" (at 60.96 113.03 0)
+    (property "LCSC" "C413002" (at 60.96 113.03 0)
       (effects (font (size 1.27 1.27)) hide)
     )
@@
       (effects (font (size 1.27 1.27)) hide)
     )
-    (property "LCSC" "" (at 67.31 113.03 0)
+    (property "LCSC" "C278580" (at 67.31 113.03 0)
       (effects (font (size 1.27 1.27)) hide)
     )
@@
       (effects (font (size 1.27 1.27)) hide)
     )
-    (property "LCSC" "" (at 73.66 113.03 0)
-      (effects (font (size 1.27 1.27)) hide)
-    )
+    (property "LCSC" "C278580" (at 73.66 113.03 0)
+      (effects (font (size 1.27 1.27)) hide)
+    )

Commit message: Switch LEDs
Parts:
- C1301, C1302: Comment Murata Electronics GRT155R61E105KE01D 1 µF ±10% 25V Ceramic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 -> (none)
- C1303, C1311: Comment Samsung Electro-Mechanics CL05A105KL5NRNC 1 µF ±10% 35V Cer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 -> (none)
- C1304, C1305, C1306, C1307, C1308, C1309, C1310, C1312, C1313, C1314: Comment Murata Electronics GRM155R62A104KE14D 0.1 µF ±10% 100V Cera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 -> (none)
- C1315, C1316: Comment KEMET C0402C150J3GACAUTO 15 pF ±5% 25V Ceramic Capacitor C0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 -> (none)
- D1301, D1302: Comment onsemi NSR20F40NXT5G Diode 40 V 2A Surface Mount 2-DSN (1.6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 -> (none)
- J1301: Comment Amphenol ICC (FCI) 10152803-00011LF USB-C (USB TYPE-C) USB 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 -> (none)
- R1301: Comment YAGEO RC0402JR-0710KL 10 kOhms ±5% 0.063W, 1/16W Chip Resis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 -> (none)
- R1302, R1303: Comment Panasonic Electronic Components ERJ-2GEJ512X 5.1 kOhms ±5% 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 -> (none)
- R1304, R1305: Comment Panasonic Electronic Components ERJ-2GEJ270X 27 Ohms ±5% 0.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 -> (none)
- R1306, R1307: Comment YAGEO RC0402FR-071KL 1 kOhms ±1% 0.063W, 1/16W Chip Resisto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 -> (none)
- SW1301: Comment Würth Elektronik 436333045822 Tactile Switch SPST-NO Side A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 -> (none)
- U1301: Comment Texas Instruments TPS73733QDRBRQ1 Linear Voltage Regulator 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 -> (none)
- U1302: Comment Raspberry Pi SC0914(13) ARM Cortex-M0+ - Microcontroller IC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 -> (none)
- U1303: Comment Winbond Electronics W25Q128JVPIQ FLASH - NOR Memory IC 128M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 -> (none)
- Y1301: Comment Abracon LLC ABM8-272-T3 12 MHz ±30ppm Crystal 10pF 50 Ohms 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 -> (none)

Commit message: Update parts based on jlcpcb availability
Parts:
- D1301, D1302: Package (none) -> 0603
- J1301: Package (none) -> USB-C-SMD
- SW1301: Package (none) -> -
- U1301: Package 8SON -> VSON-8-EP(3x3)
- U1302: Package 56QFN -> QFN-56(7x7)
- U1303: Package 8WSON -> WSON-8-EP(5x6)
- Y1301: Package (none) -> SMD3225-4P
Changed lines of the file:
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@@
+      (effects (font (size 1.27 1.27)) hide)
+    )
+    (property "Package" "-" (at 256.54 128.27 0)
       (effects (font (size 1.27 1.27)) hide)
     )
@@
       (effects (font (size 1.27 1.27)) hide)
     )
+    (property "Package" "0603" (at 66.04 36.83 0)
+      (effects (font (size 1.27 1.27)) hide)
+    )
     (pin "2")
     (pin "1")
@@
     )
     (property "LCSC" "C5410523" (at 31.75 100.33 0)
+      (effects (font (size 1.27 1.27)) hide)
+    )
+    (property "Package" "USB-C-SMD" (at 31.75 100.33 0)
       (effects (font (size 1.27 1.27)) hide)
     )
@@
       (effects (font (size 1.27 1.27)) hide)
     )
+    (property "Package" "0603" (at 66.04 43.18 0)
+      (effects (font (size 1.27 1.27)) hide)
+    )
     (pin "2")
     (pin "1")
@@
       (effects (font (size 1.27 1.27)) hide)
     )
-    (property "Package" " 8SON" (at 119.38 30.48 0)
+    (property "Package" "VSON-8-EP(3x3)" (at 119.38 30.48 0)
       (effects (font (size 1.27 1.27)) hide)
     )
@@
       (effects (font (size 1.27 1.27)) hide)
     )
-    (property "Package" " 8WSON" (at 233.68 142.24 0)
+    (property "Package" "WSON-8-EP(5x6)" (at 233.68 142.24 0)
       (effects (font (size 1.27 1.27)) hide)
     )
@@
       (effects (font (size 1.27 1.27)) hide)
     )
-    (property "Package" " 56QFN" (at 121.92 120.65 0)
+    (property "Package" "QFN-56(7x7)" (at 121.92 120.65 0)
       (effects (font (size 1.27 1.27)) hide)
     )
@@
       (effects (font (size 1.27 1.27)) hide)
     )
+    (property "Package" "SMD3225-4P" (at 39.37 157.48 0)
+      (effects (font (size 1.27 1.27)) hide)
+    )

Commit message: Update rp2040 jlcpcb part number
Parts:
- U1302: LCSC C3227924 -> C2040; Manufacturer Part Number SC0914(13) -> RP2040
Changed lines of the file:
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@@
       (effects (font (size 1.27 1.27)) hide)
     )
-    (property "Manufacturer Part Number" "SC0914(13)" (at 121.92 120.65 0)
+    (property "Manufacturer Part Number" "RP2040" (at 121.92 120.65 0)
       (effects (font (size 1.27 1.27)) hide)
     )
@@
       (effects (font (size 1.27 1.27)) hide)
     )
-    (property "LCSC" "C3227924" (at 121.92 120.65 0)
+    (property "LCSC" "C2040" (at 121.92 120.65 0)
       (effects (font (size 1.27 1.27)) hide)
     )
