File: stepper-interface/tmc5160.kicad_sch (KiCad schematic)
At the start: 30 parts, among them J401 Molex_Pico-SPOX_Horizontal, J402 Molex_Pico-Clasp_Horizontal, U401 TMC5160A-WA, U402 MAX6816, X401 16MHz

Commit message: Use jlcpcb part number
Parts:
- R404, R405: LCSC C4090676 -> C2683383; Manufacturer Delta Electronics/Cyntec -> TA-I Tech; Manufacturer Part Number VSRP1206S1-R150F -> RLH12FTCR150; Synopsis RES 0.15 OHM 1% 1W -> 1W 150m Surface Mount Current Sensing Resistor; Vendor Digi-Key -> JLCPCB; Vendor Part Number 2037-VSRP1206S1-R150FCT-ND -> C2683383
Changed lines of the file:
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@@
       (effects (font (size 0.762 0.762)))
     )
-    (property "Vendor" "Digi-Key" (at 111.252 118.11 90)
-      (effects (font (size 1.524 1.524)) hide)
-    )
-    (property "Vendor Part Number" "2037-VSRP1206S1-R150FCT-ND" (at 113.792 115.57 90)
+    (property "Vendor" "JLCPCB" (at 111.252 118.11 90)
+      (effects (font (size 1.524 1.524)) hide)
+    )
+    (property "Vendor Part Number" "C2683383" (at 113.792 115.57 90)
       (effects (font (size 1.524 1.524)) hide)
     )
@@
       (effects (font (size 1.27 1.27)) hide)
     )
-    (property "Manufacturer" "Delta Electronics/Cyntec" (at 106.68 120.65 0)
-      (effects (font (size 1.27 1.27)) hide)
-    )
-    (property "Manufacturer Part Number" "VSRP1206S1-R150F" (at 106.68 120.65 0)
-      (effects (font (size 1.27 1.27)) hide)
-    )
-    (property "Synopsis" "RES 0.15 OHM 1% 1W" (at 116.332 113.03 90)
-      (effects (font (size 1.524 1.524)) hide)
-    )
-    (property "LCSC" "C4090676" (at 106.68 120.65 0)
+    (property "Manufacturer" "TA-I Tech" (at 106.68 120.65 0)
+      (effects (font (size 1.27 1.27)) hide)
+    )
+    (property "Manufacturer Part Number" "RLH12FTCR150" (at 106.68 120.65 0)
+      (effects (font (size 1.27 1.27)) hide)
+    )
+    (property "Synopsis" "1W 150m Surface Mount Current Sensing Resistor" (at 116.332 113.03 90)
+      (effects (font (size 1.524 1.524)) hide)
+    )
+    (property "LCSC" "C2683383" (at 106.68 120.65 0)
       (effects (font (size 1.27 1.27)) hide)
     )
@@
       (effects (font (size 0.762 0.762)))
     )
-    (property "Vendor" "Digi-Key" (at 141.732 118.11 90)
-      (effects (font (size 1.524 1.524)) hide)
-    )
-    (property "Vendor Part Number" "2037-VSRP1206S1-R150FCT-ND" (at 144.272 115.57 90)
+    (property "Vendor" "JLCPCB" (at 141.732 118.11 90)
+      (effects (font (size 1.524 1.524)) hide)
+    )
+    (property "Vendor Part Number" "C2683383" (at 144.272 115.57 90)
       (effects (font (size 1.524 1.524)) hide)
     )
@@
       (effects (font (size 1.27 1.27)) hide)
     )
-    (property "Manufacturer" "Delta Electronics/Cyntec" (at 137.16 120.65 0)
-      (effects (font (size 1.27 1.27)) hide)
-    )
-    (property "Manufacturer Part Number" "VSRP1206S1-R150F" (at 137.16 120.65 0)
-      (effects (font (size 1.27 1.27)) hide)
-    )
-    (property "Synopsis" "RES 0.15 OHM 1% 1W" (at 146.812 113.03 90)
-      (effects (font (size 1.524 1.524)) hide)
-    )
-    (property "LCSC" "C4090676" (at 137.16 120.65 0)
-      (effects (font (size 1.27 1.27)) hide)
-    )
+    (property "Manufacturer" "TA-I Tech" (at 137.16 120.65 0)
+      (effects (font (size 1.27 1.27)) hide)
+    )
+    (property "Manufacturer Part Number" "RLH12FTCR150" (at 137.16 120.65 0)
+      (effects (font (size 1.27 1.27)) hide)
+    )
+    (property "Synopsis" "1W 150m Surface Mount Current Sensing Resistor" (at 146.812 113.03 90)
+      (effects (font (size 1.524 1.524)) hide)
+    )
+    (property "LCSC" "C2683383" (at 137.16 120.65 0)
+      (effects (font (size 1.27 1.27)) hide)
+    )
