File: tmc5160-usb/mosfet.kicad_sch (KiCad schematic)
At the start: 2 parts, among them U501 BUK7D36-60EX

Commit message: stepper-interface -> tmc5160-usb
Other:
- title: stepper-interface -> tmc5160-usb
Changed lines of the file:
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@@
   (paper "A4")
   (title_block
-    (title "stepper-interface")
+    (title "tmc5160-usb")
     (date "2024-05-10")
     (rev "1.0")
@@
     (pin "8")
     (instances
-      (project "stepper-interface"
+      (project "tmc5160-usb"
         (path "/df2b2e89-e055-4140-95de-f1df723db034/039ac378-5273-4081-85bf-9eb26cb5ed57/166b4ba4-5822-49d8-b309-f52ce04f60b1"
           (reference "U501") (unit 1)
@@
     (pin "1")
     (instances
-      (project "stepper-interface"
+      (project "tmc5160-usb"
         (path "/df2b2e89-e055-4140-95de-f1df723db034/039ac378-5273-4081-85bf-9eb26cb5ed57/166b4ba4-5822-49d8-b309-f52ce04f60b1"
           (reference "R501") (unit 1)
