File: tmc5160-usb/power.kicad_sch (KiCad schematic)
At the start: 18 parts, among them J301 Molex_Pico-SPOX_Horizontal, J302 Molex_Pico-Lock-PLUS_Vertical, M301 Fan_5VDC_25x25x8mm, Q301 MOSFET-N-CH, U301 Switching_5V_500mA, U302 Linear_3.3V_1A

Commit message: stepper-interface -> tmc5160-usb
Other:
- title: stepper-interface -> tmc5160-usb
Changed lines of the file:
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@@
   (paper "A4")
   (title_block
-    (title "stepper-interface")
+    (title "tmc5160-usb")
     (date "2024-05-10")
     (rev "1.0")
@@
     (pin "1")
     (instances
-      (project "stepper-interface"
+      (project "tmc5160-usb"
         (path "/df2b2e89-e055-4140-95de-f1df723db034/c1dd8f61-494c-402f-8e59-08309c64fc3f"
           (reference "D303") (unit 1)
@@
     (pin "7")
     (instances
-      (project "stepper-interface"
+      (project "tmc5160-usb"
         (path "/df2b2e89-e055-4140-95de-f1df723db034/c1dd8f61-494c-402f-8e59-08309c64fc3f"
           (reference "U302") (unit 1)
@@
     (pin "1")
     (instances
-      (project "stepper-interface"
+      (project "tmc5160-usb"
         (path "/df2b2e89-e055-4140-95de-f1df723db034/c1dd8f61-494c-402f-8e59-08309c64fc3f"
           (reference "#FLG0303") (unit 1)
@@
     (pin "1")
     (instances
-      (project "stepper-interface"
+      (project "tmc5160-usb"
         (path "/df2b2e89-e055-4140-95de-f1df723db034/c1dd8f61-494c-402f-8e59-08309c64fc3f"
           (reference "J302") (unit 1)
@@
     (pin "1")
     (instances
-      (project "stepper-interface"
+      (project "tmc5160-usb"
         (path "/df2b2e89-e055-4140-95de-f1df723db034/c1dd8f61-494c-402f-8e59-08309c64fc3f"
           (reference "C302") (unit 1)
@@
     (pin "1")
     (instances
-      (project "stepper-interface"
+      (project "tmc5160-usb"
         (path "/df2b2e89-e055-4140-95de-f1df723db034/c1dd8f61-494c-402f-8e59-08309c64fc3f"
           (reference "L301") (unit 1)
@@
     (pin "1")
     (instances
-      (project "stepper-interface"
+      (project "tmc5160-usb"
         (path "/df2b2e89-e055-4140-95de-f1df723db034/c1dd8f61-494c-402f-8e59-08309c64fc3f"
           (reference "R303") (unit 1)
@@
     (pin "1")
     (instances
-      (project "stepper-interface"
+      (project "tmc5160-usb"
         (path "/df2b2e89-e055-4140-95de-f1df723db034/c1dd8f61-494c-402f-8e59-08309c64fc3f"
           (reference "J301") (unit 1)
@@
     (pin "1")
     (instances
-      (project "stepper-interface"
+      (project "tmc5160-usb"
         (path "/df2b2e89-e055-4140-95de-f1df723db034/c1dd8f61-494c-402f-8e59-08309c64fc3f"
           (reference "C304") (unit 1)
@@
     (pin "1")
     (instances
-      (project "stepper-interface"
+      (project "tmc5160-usb"
         (path "/df2b2e89-e055-4140-95de-f1df723db034/c1dd8f61-494c-402f-8e59-08309c64fc3f"
           (reference "C301") (unit 1)
@@
     (pin "1")
     (instances
-      (project "stepper-interface"
+      (project "tmc5160-usb"
         (path "/df2b2e89-e055-4140-95de-f1df723db034/c1dd8f61-494c-402f-8e59-08309c64fc3f"
           (reference "D301") (unit 1)
@@
     (pin "1")
     (instances
-      (project "stepper-interface"
+      (project "tmc5160-usb"
         (path "/df2b2e89-e055-4140-95de-f1df723db034/c1dd8f61-494c-402f-8e59-08309c64fc3f"
           (reference "D302") (unit 1)
@@
     (pin "1")
     (instances
-      (project "stepper-interface"
+      (project "tmc5160-usb"
         (path "/df2b2e89-e055-4140-95de-f1df723db034/c1dd8f61-494c-402f-8e59-08309c64fc3f"
           (reference "C305") (unit 1)
@@
     (pin "1")
     (instances
-      (project "stepper-interface"
+      (project "tmc5160-usb"
         (path "/df2b2e89-e055-4140-95de-f1df723db034/c1dd8f61-494c-402f-8e59-08309c64fc3f"
           (reference "#FLG0302") (unit 1)
@@
     (pin "2")
     (instances
-      (project "stepper-interface"
+      (project "tmc5160-usb"
         (path "/df2b2e89-e055-4140-95de-f1df723db034/c1dd8f61-494c-402f-8e59-08309c64fc3f"
           (reference "R302") (unit 1)
@@
     (pin "1")
     (instances
-      (project "stepper-interface"
+      (project "tmc5160-usb"
         (path "/df2b2e89-e055-4140-95de-f1df723db034/c1dd8f61-494c-402f-8e59-08309c64fc3f"
           (reference "#FLG0301") (unit 1)
@@
     (pin "1")
     (instances
-      (project "stepper-interface"
+      (project "tmc5160-usb"
         (path "/df2b2e89-e055-4140-95de-f1df723db034/c1dd8f61-494c-402f-8e59-08309c64fc3f"
           (reference "R301") (unit 1)
@@
     (pin "4")
     (instances
-      (project "stepper-interface"
+      (project "tmc5160-usb"
         (path "/df2b2e89-e055-4140-95de-f1df723db034/c1dd8f61-494c-402f-8e59-08309c64fc3f"
           (reference "U301") (unit 1)
@@
     (pin "3")
     (instances
-      (project "stepper-interface"
+      (project "tmc5160-usb"
         (path "/df2b2e89-e055-4140-95de-f1df723db034/c1dd8f61-494c-402f-8e59-08309c64fc3f"
           (reference "Q301") (unit 1)
@@
     (pin "2")
     (instances
-      (project "stepper-interface"
+      (project "tmc5160-usb"
         (path "/df2b2e89-e055-4140-95de-f1df723db034/c1dd8f61-494c-402f-8e59-08309c64fc3f"
           (reference "M301") (unit 1)
@@
     (pin "1")
     (instances
-      (project "stepper-interface"
+      (project "tmc5160-usb"
         (path "/df2b2e89-e055-4140-95de-f1df723db034/c1dd8f61-494c-402f-8e59-08309c64fc3f"
           (reference "C303") (unit 1)
