File: tmc5160-usb/rp2040.kicad_sch (KiCad schematic)
At the start: 31 parts, among them J1301 Connector_USB_C_Receptacle, SW1301 Switch_Tactile_SPST-NO_SMT_Si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, U1301 Linear_3.3V_1A, U1302 MCU_RP2040, U1303 Memory_Flash_W25Q128JVZPIQ, Y1301 Crystal_12MHz

Commit message: stepper-interface -> tmc5160-usb
Other:
- title: stepper-interface -> tmc5160-usb
Changed lines of the file:
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@@
   (paper "A4")
   (title_block
-    (title "stepper-interface")
+    (title "tmc5160-usb")
     (date "2024-05-10")
     (rev "1.0")
@@
     (pin "2")
     (instances
-      (project "stepper-interface"
+      (project "tmc5160-usb"
         (path "/df2b2e89-e055-4140-95de-f1df723db034/69dff8eb-dcc1-4f17-9e1d-cf8103035e92"
           (reference "R1306") (unit 1)
@@
     (pin "1")
     (instances
-      (project "stepper-interface"
+      (project "tmc5160-usb"
         (path "/df2b2e89-e055-4140-95de-f1df723db034/69dff8eb-dcc1-4f17-9e1d-cf8103035e92"
           (reference "C1311") (unit 1)
@@
     (pin "1")
     (instances
-      (project "stepper-interface"
+      (project "tmc5160-usb"
         (path "/df2b2e89-e055-4140-95de-f1df723db034/69dff8eb-dcc1-4f17-9e1d-cf8103035e92"
           (reference "C1316") (unit 1)
@@
     (pin "1")
     (instances
-      (project "stepper-interface"
+      (project "tmc5160-usb"
         (path "/df2b2e89-e055-4140-95de-f1df723db034/69dff8eb-dcc1-4f17-9e1d-cf8103035e92"
           (reference "C1307") (unit 1)
@@
     (pin "1")
     (instances
-      (project "stepper-interface"
+      (project "tmc5160-usb"
         (path "/df2b2e89-e055-4140-95de-f1df723db034/69dff8eb-dcc1-4f17-9e1d-cf8103035e92"
           (reference "C1309") (unit 1)
@@
     (pin "1")
     (instances
-      (project "stepper-interface"
+      (project "tmc5160-usb"
         (path "/df2b2e89-e055-4140-95de-f1df723db034/69dff8eb-dcc1-4f17-9e1d-cf8103035e92"
           (reference "C1313") (unit 1)
@@
     (pin "2")
     (instances
-      (project "stepper-interface"
+      (project "tmc5160-usb"
         (path "/df2b2e89-e055-4140-95de-f1df723db034/69dff8eb-dcc1-4f17-9e1d-cf8103035e92"
           (reference "SW1301") (unit 1)
@@
     (pin "1")
     (instances
-      (project "stepper-interface"
+      (project "tmc5160-usb"
         (path "/df2b2e89-e055-4140-95de-f1df723db034/69dff8eb-dcc1-4f17-9e1d-cf8103035e92"
           (reference "#FLG01301") (unit 1)
@@
     (pin "1")
     (instances
-      (project "stepper-interface"
+      (project "tmc5160-usb"
         (path "/df2b2e89-e055-4140-95de-f1df723db034/69dff8eb-dcc1-4f17-9e1d-cf8103035e92"
           (reference "C1304") (unit 1)
@@
     (pin "1")
     (instances
-      (project "stepper-interface"
+      (project "tmc5160-usb"
         (path "/df2b2e89-e055-4140-95de-f1df723db034/69dff8eb-dcc1-4f17-9e1d-cf8103035e92"
           (reference "C1306") (unit 1)
@@
     (pin "1")
     (instances
-      (project "stepper-interface"
+      (project "tmc5160-usb"
         (path "/df2b2e89-e055-4140-95de-f1df723db034/69dff8eb-dcc1-4f17-9e1d-cf8103035e92"
           (reference "D1301") (unit 1)
@@
     (pin "1")
     (instances
-      (project "stepper-interface"
+      (project "tmc5160-usb"
         (path "/df2b2e89-e055-4140-95de-f1df723db034/69dff8eb-dcc1-4f17-9e1d-cf8103035e92"
           (reference "C1314") (unit 1)
@@
     (pin "1")
     (instances
-      (project "stepper-interface"
+      (project "tmc5160-usb"
         (path "/df2b2e89-e055-4140-95de-f1df723db034/69dff8eb-dcc1-4f17-9e1d-cf8103035e92"
           (reference "C1301") (unit 1)
@@
     (pin "2")
     (instances
-      (project "stepper-interface"
+      (project "tmc5160-usb"
         (path "/df2b2e89-e055-4140-95de-f1df723db034/69dff8eb-dcc1-4f17-9e1d-cf8103035e92"
           (reference "R1302") (unit 1)
@@
     (pin "1")
     (instances
-      (project "stepper-interface"
+      (project "tmc5160-usb"
         (path "/df2b2e89-e055-4140-95de-f1df723db034/69dff8eb-dcc1-4f17-9e1d-cf8103035e92"
           (reference "C1310") (unit 1)
@@
     (pin "1")
     (instances
-      (project "stepper-interface"
+      (project "tmc5160-usb"
         (path "/df2b2e89-e055-4140-95de-f1df723db034/69dff8eb-dcc1-4f17-9e1d-cf8103035e92"
           (reference "C1312") (unit 1)
@@
     (pin "1")
     (instances
-      (project "stepper-interface"
+      (project "tmc5160-usb"
         (path "/df2b2e89-e055-4140-95de-f1df723db034/69dff8eb-dcc1-4f17-9e1d-cf8103035e92"
           (reference "C1305") (unit 1)
@@
     (pin "2")
     (instances
-      (project "stepper-interface"
+      (project "tmc5160-usb"
         (path "/df2b2e89-e055-4140-95de-f1df723db034/69dff8eb-dcc1-4f17-9e1d-cf8103035e92"
           (reference "R1303") (unit 1)
@@
     (pin "1")
     (instances
-      (project "stepper-interface"
+      (project "tmc5160-usb"
         (path "/df2b2e89-e055-4140-95de-f1df723db034/69dff8eb-dcc1-4f17-9e1d-cf8103035e92"
           (reference "C1302") (unit 1)
@@
     (pin "1")
     (instances
-      (project "stepper-interface"
+      (project "tmc5160-usb"
         (path "/df2b2e89-e055-4140-95de-f1df723db034/69dff8eb-dcc1-4f17-9e1d-cf8103035e92"
           (reference "C1308") (unit 1)
@@
     (pin "S4")
     (instances
-      (project "stepper-interface"
+      (project "tmc5160-usb"
         (path "/df2b2e89-e055-4140-95de-f1df723db034/69dff8eb-dcc1-4f17-9e1d-cf8103035e92"
           (reference "J1301") (unit 1)
@@
     (pin "1")
     (instances
-      (project "stepper-interface"
+      (project "tmc5160-usb"
         (path "/df2b2e89-e055-4140-95de-f1df723db034/69dff8eb-dcc1-4f17-9e1d-cf8103035e92"
           (reference "D1302") (unit 1)
@@
     (pin "2")
     (instances
-      (project "stepper-interface"
+      (project "tmc5160-usb"
         (path "/df2b2e89-e055-4140-95de-f1df723db034/69dff8eb-dcc1-4f17-9e1d-cf8103035e92"
           (reference "U1301") (unit 1)
@@
     (pin "1")
     (instances
-      (project "stepper-interface"
+      (project "tmc5160-usb"
         (path "/df2b2e89-e055-4140-95de-f1df723db034/69dff8eb-dcc1-4f17-9e1d-cf8103035e92"
           (reference "U1303") (unit 1)
@@
     (pin "1")
     (instances
-      (project "stepper-interface"
+      (project "tmc5160-usb"
         (path "/df2b2e89-e055-4140-95de-f1df723db034/69dff8eb-dcc1-4f17-9e1d-cf8103035e92"
           (reference "R1304") (unit 1)
@@
     (pin "6")
     (instances
-      (project "stepper-interface"
+      (project "tmc5160-usb"
         (path "/df2b2e89-e055-4140-95de-f1df723db034/69dff8eb-dcc1-4f17-9e1d-cf8103035e92"
           (reference "U1302") (unit 1)
@@
     (pin "1")
     (instances
-      (project "stepper-interface"
+      (project "tmc5160-usb"
         (path "/df2b2e89-e055-4140-95de-f1df723db034/69dff8eb-dcc1-4f17-9e1d-cf8103035e92"
           (reference "C1315") (unit 1)
@@
     (pin "1")
     (instances
-      (project "stepper-interface"
+      (project "tmc5160-usb"
         (path "/df2b2e89-e055-4140-95de-f1df723db034/69dff8eb-dcc1-4f17-9e1d-cf8103035e92"
           (reference "C1303") (unit 1)
@@
     (pin "2")
     (instances
-      (project "stepper-interface"
+      (project "tmc5160-usb"
         (path "/df2b2e89-e055-4140-95de-f1df723db034/69dff8eb-dcc1-4f17-9e1d-cf8103035e92"
           (reference "R1307") (unit 1)
@@
     (pin "2")
     (instances
-      (project "stepper-interface"
+      (project "tmc5160-usb"
         (path "/df2b2e89-e055-4140-95de-f1df723db034/69dff8eb-dcc1-4f17-9e1d-cf8103035e92"
           (reference "R1301") (unit 1)
@@
     (pin "1")
     (instances
-      (project "stepper-interface"
+      (project "tmc5160-usb"
         (path "/df2b2e89-e055-4140-95de-f1df723db034/69dff8eb-dcc1-4f17-9e1d-cf8103035e92"
           (reference "R1305") (unit 1)
@@
     (pin "3")
     (instances
-      (project "stepper-interface"
+      (project "tmc5160-usb"
         (path "/df2b2e89-e055-4140-95de-f1df723db034/69dff8eb-dcc1-4f17-9e1d-cf8103035e92"
           (reference "Y1301") (unit 1)
