File: tmc5160-usb/rp2040.kicad_sch (KiCad schematic)
At the start: 31 parts, among them J1301 Connector_USB_C_Receptacle, SW1301 Switch_Tactile_SPST-NO_SMT_Si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, U1301 Linear_3.3V_1A, U1302 MCU_RP2040, U1303 Memory_Flash_W25Q128JVZPIQ, Y1301 Crystal_12MHz

Commit message: mosi -> copi, miso -> cipo
Connections:
- net MISO renamed CIPO
- net MOSI renamed COPI
Changed lines of the file:
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@@
     (effects (font (size 1.27 1.27)) (justify right bottom))
   )
-  (label "MISO" (at 149.86 133.35 0) (fields_autoplaced)
+  (label "CIPO" (at 149.86 133.35 0) (fields_autoplaced)
     (effects (font (size 1.27 1.27)) (justify left bottom))
   )
@@
     (effects (font (size 1.27 1.27)) (justify right bottom))
   )
-  (label "MISO" (at 40.64 40.64 0) (fields_autoplaced)
+  (label "CIPO" (at 40.64 40.64 0) (fields_autoplaced)
     (effects (font (size 1.27 1.27)) (justify left bottom))
   )
@@
     (effects (font (size 1.27 1.27)) (justify right bottom))
   )
-  (label "MOSI" (at 40.64 38.1 0) (fields_autoplaced)
+  (label "COPI" (at 40.64 38.1 0) (fields_autoplaced)
     (effects (font (size 1.27 1.27)) (justify left bottom))
   )
@@
     (effects (font (size 1.27 1.27)) (justify right bottom))
   )
-  (label "MOSI" (at 149.86 130.81 0) (fields_autoplaced)
+  (label "COPI" (at 149.86 130.81 0) (fields_autoplaced)
     (effects (font (size 1.27 1.27)) (justify left bottom))
   )
@@
     (effects (font (size 1.27 1.27)) (justify right))
   )
-  (hierarchical_label "MISO" (shape input) (at 38.1 40.64 180) (fields_autoplaced)
-    (effects (font (size 1.27 1.27)) (justify right))
-  )
-  (hierarchical_label "MOSI" (shape output) (at 38.1 38.1 180) (fields_autoplaced)
-    (effects (font (size 1.27 1.27)) (justify right))
-  )
+  (hierarchical_label "CIPO" (shape input) (at 38.1 40.64 180) (fields_autoplaced)
+    (effects (font (size 1.27 1.27)) (justify right))
+  )
+  (hierarchical_label "COPI" (shape output) (at 38.1 38.1 180) (fields_autoplaced)
+    (effects (font (size 1.27 1.27)) (justify right))
+  )
