File: tmc5160-usb/tmc5160-usb.kicad_sch (KiCad schematic)
At the start: 0 parts

Commit message: stepper-interface -> tmc5160-usb
Other:
- title: stepper-interface -> tmc5160-usb
Changed lines of the file:
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@@
   (paper "A4")
   (title_block
-    (title "stepper-interface")
+    (title "tmc5160-usb")
     (date "2024-05-10")
     (rev "1.0")
@@
     )
     (instances
-      (project "stepper-interface"
+      (project "tmc5160-usb"
         (path "/df2b2e89-e055-4140-95de-f1df723db034" (page "4"))
       )
@@
     )
     (instances
-      (project "stepper-interface"
+      (project "tmc5160-usb"
         (path "/df2b2e89-e055-4140-95de-f1df723db034" (page "2"))
       )
@@
     )
     (instances
-      (project "stepper-interface"
+      (project "tmc5160-usb"
         (path "/df2b2e89-e055-4140-95de-f1df723db034" (page "13"))
       )
@@
     )
     (instances
-      (project "stepper-interface"
+      (project "tmc5160-usb"
         (path "/df2b2e89-e055-4140-95de-f1df723db034" (page "3"))
       )
