File: tmc5160-usb/tmc5160-usb.kicad_sch (KiCad schematic)
At the start: 0 parts

Commit message: mosi -> copi, miso -> cipo
Other:
- sheet rp2040 ports: added CIPO, COPI; removed MISO, MOSI
- sheet tmc5160 ports: added CIPO, COPI; removed MISO, MOSI
Changed lines of the file:
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@@
     (effects (font (size 1.27 1.27)) (justify left bottom))
   )
-  (label "MOSI" (at 128.27 130.81 180) (fields_autoplaced)
+  (label "COPI" (at 128.27 130.81 180) (fields_autoplaced)
     (effects (font (size 1.27 1.27)) (justify right bottom))
   )
@@
     (effects (font (size 1.27 1.27)) (justify left bottom))
   )
-  (label "MISO" (at 128.27 97.79 180) (fields_autoplaced)
+  (label "CIPO" (at 128.27 97.79 180) (fields_autoplaced)
     (effects (font (size 1.27 1.27)) (justify right bottom))
   )
@@
     (effects (font (size 1.27 1.27)) (justify right bottom))
   )
-  (label "MOSI" (at 154.94 97.79 0) (fields_autoplaced)
+  (label "COPI" (at 154.94 97.79 0) (fields_autoplaced)
     (effects (font (size 1.27 1.27)) (justify left bottom))
   )
@@
     (effects (font (size 1.27 1.27)) (justify right bottom))
   )
-  (label "MISO" (at 154.94 125.73 0) (fields_autoplaced)
+  (label "CIPO" (at 154.94 125.73 0) (fields_autoplaced)
     (effects (font (size 1.27 1.27)) (justify left bottom))
   )
@@
       (effects (font (size 1.27 1.27)) (justify right))
     )
-    (pin "MISO" output (at 152.4 125.73 0)
+    (pin "CIPO" output (at 152.4 125.73 0)
       (effects (font (size 1.27 1.27)) (justify right))
     )
-    (pin "MOSI" input (at 130.81 130.81 180)
+    (pin "COPI" input (at 130.81 130.81 180)
       (effects (font (size 1.27 1.27)) (justify left))
     )
@@
       (effects (font (size 1.27 1.27)) (justify right))
     )
-    (pin "MOSI" output (at 152.4 97.79 0)
+    (pin "COPI" output (at 152.4 97.79 0)
       (effects (font (size 1.27 1.27)) (justify right))
     )
-    (pin "MISO" input (at 130.81 97.79 180)
+    (pin "CIPO" input (at 130.81 97.79 180)
       (effects (font (size 1.27 1.27)) (justify left))
     )
